File: CM4_GPIO.kicad_sch (KiCad schematic)
At the start: 21 parts, among them IC5 74LVC1G07QSE-7, J3 THD-20-R, SW1 SW_Push, SW2 SW_Push, SW3 SW_DPDT_x2, SW4 SW_DPDT_x2

Commit message: think im done with schematic
Parts:
- added SW5: SW_Push, symbol Switch:SW_Push
Connections:
- net GND: now also SW5.1
- net GPIO3: now also SW5.2
Other:
- note added: "Hard Reset Button"
- note added: "Press for >1 ms and then release to send a shutdown signal and safely shutdown."
- note added: "Soft Reset Button"
- note removed: "CM4 Reset Button"
- moved on the sheet: D2, IC5, J3, R4, TP2
