File: HDMI.kicad_sch (KiCad schematic)
At the start: 5 parts, among them J9 HDMI_E, U5 RT9742SNGV

Commit message: think im done with schematic
Parts:
- removed C1, C2: 100n, Capacitor_SMD:C_0402_1005Metric, symbol Device:C
- removed U5: RT9742SNGV, symbol CM4IO:RT9742SNGV
- added C43, C45: 100 n, Capacitor_SMD:C_0402_1005Metric, symbol Device:C
- added C44: 100n, Capacitor_SMD:C_0402_1005Metric, symbol Device:C
- added IC6: TPS2553QDBVRQ1, SOT95P280X145-6N, symbol TPS2553QDBVRQ1:TPS2553QDBVRQ1
- added R27: 100 n, symbol Device:R
- added R28: 80 k, symbol Device:R
Connections:
- net +5V_PWR: now also C43.1, IC6.1 (IN)
- net GND: now also C43.2, C44.2, C45.2, IC6.2 (GND), R28.1
- net HDMI_5v: now also C44.1, IC6.6 (OUT)
- new net: C45.1, IC6.3 (EN), IC6.4 (nFAULT), R27.2
- new net: IC6.5 (ILIM), R28.2
- new net GLOBAL_EN: R27.1
Other:
- note added: "Limit at 300-350 mA"
