File: HDMI.kicad_sch (KiCad schematic)
At the start: 23 parts, among them IC8 TPS2557QDRBTQ1, IC9 TPS2557QDRBTQ1, J13 USB_C_Receptacle_USB2.0_16P, J7 USB_C_Receptacle

Commit message: rrrrrrrr
Parts:
- removed C15: 120uF, Capacitor_SMD:C_0603_1608Metric, symbol Device:C
- removed C21, C28, C32, C33: 100n, Capacitor_SMD:C_0603_1608Metric, symbol Device:C
- removed D15, D18: TPD4E05U06DQAR, Controls_Pi:DQA_R-PUSON-N10_, symbol TPD4E05U06DQAR:TPD4E05U06DQAR
- removed D6: VBUS_PWR LED, LED_SMD:LED_0603_1608Metric, symbol Device:LED
- removed FB3, FB5: FerriteBead, Inductor_SMD:L_1206_3216Metric, symbol Device:FerriteBead
- removed IC9: TPS2557QDRBTQ1, SON65P300X300X100-9N-D, symbol TPS2557QDRBTQ1:TPS2557QDRBTQ1
- removed J13: USB_C_Receptacle_USB2.0_16P, Connector_USB:USB_C_Receptacle_GCT_USB4105-xx-A_16P_TopMnt_Horizontal, symbol Connector:USB_C_Receptacle_USB2.0_16P
- removed J7: USB_C_Receptacle, symbol Connector:USB_C_Receptacle
- removed Module2: ComputeModule5-CM5, CM5IO:Raspberry-Pi-5-Compute-Module, symbol CM5IO:ComputeModule5-CM5
- removed R16, R21: 56k, Resistor_SMD:R_0603_1608Metric, symbol Device:R
- removed R18: 1.5k, Resistor_SMD:R_0603_1608Metric, symbol Device:R
- removed R29: 120k, Resistor_SMD:R_0603_1608Metric, symbol Device:R
- removed R41: 20k, Resistor_SMD:R_0603_1608Metric, symbol Device:R
- added C29: 100uF, Capacitor_SMD:C_0805_2012Metric, symbol Device:C
- added D10, D11: TPD4E05U06DQAR, Controls_Pi:DQA_R-PUSON-N10_, symbol TPD4E05U06DQAR:TPD4E05U06DQAR
- added J9: HDMI_E, Controls_Pi:MX50019NQ1, symbol Connector:HDMI_E
- added R23: 100k, Resistor_SMD:R_0603_1608Metric, symbol Device:R
- R26: value 100k -> 180k
Connections:
- net CC1 is gone; now on net HDMI0_CEC: D17.1 (D1+), D17.10 (NC_4)
- net CC2 is gone; now on net HDMI0_HOTPLUG: D17.2 (D1-), D17.9 (NC_3)
- net USB_PWR_D+ is gone; now on net HDMI0_SDA: D17.5 (D2-), D17.6 (NC_1)
- net USB_PWR_D- is gone; now on net HDMI0_SCL: D17.4 (D2+), D17.7 (NC_2)
- net VBUS_Hub is gone; now on net +5V: IC8.2 (IN_1)
- net +5V: now also C16.1; no longer IC8.6 (OUT_1)
- net GLOBAL_EN: now also R23.1; no longer R26.2
- net GND: now also R26.2, C29.2, D10.3 (GND_1), D10.8 (GND_2), D11.3 (GND_1), D11.8 (GND_2), J9.11 (CKS), J9.17 (GND), J9.2 (D2S), J9.5 (D1S), J9.8 (D0S), J9.SH
- net HDMI0_CEC: now also J9.13 (CEC)
- net HDMI0_CK_N: now also D11.2 (D1-), D11.9 (NC_3), J9.12 (CK-)
- net HDMI0_CK_P: now also D11.1 (D1+), D11.10 (NC_4), J9.10 (CK+)
- net HDMI0_D0_N: now also D10.5 (D2-), D10.6 (NC_1), J9.9 (D0-)
- net HDMI0_D0_P: now also D10.4 (D2+), D10.7 (NC_2), J9.7 (D0+)
- net HDMI0_D1_N: now also D11.5 (D2-), D11.6 (NC_1), J9.6 (D1-)
- net HDMI0_D1_P: now also D11.4 (D2+), D11.7 (NC_2), J9.4 (D1+)
- net HDMI0_D2_N: now also D10.2 (D1-), D10.9 (NC_3), J9.3 (D2-)
- net HDMI0_D2_P: now also D10.1 (D1+), D10.10 (NC_4), J9.1 (D2+)
- net HDMI0_HOTPLUG: now also J9.19 (HPD)
- net HDMI0_SCL: now also J9.15 (SCL)
- net HDMI0_SDA: now also J9.16 (SDA)
- net at IC8.4 (EN): now also R23.2; no longer R26.1
- net at IC8.5 (ILIM): now also R26.1
- new net HDMI_5V: C29.1, IC8.6 (OUT_1), J9.18 (+5V)
- no-connect marks 60 -> 4
Other:
- removed sheet all_usb
- removed sheet hdmi_protected
- note added: "Added this"
- note added: "Current lim and rpp"
- note added: "ESD Protection Diodes"
- note added: "Ilim: ~500mA"
- note removed: "CM5 negotiates pwr thru CC1/2"
- note removed: "ESD"
- note removed: "HUB"
- note removed: "High speed pins"
- note removed: "Ilim: ~5A"
- note removed: "Ilim: ~900mA"
- note removed: "PWR"
- note removed: "Set so that USB can provide 5V/5A to pi"
- note removed: "USB C Power Port"
- note removed: "USB_OTG needs to be pulled low when connected to debug Pull high otherwise"
- note removed: "VBUS -> 5V"
