File: PiBoard.kicad_sch (KiCad schematic)
At the start: 0 parts

Commit message: think im done with schematic
Other:
- sheet HDMI and High Speed ports: added GLOBAL_EN; removed none
Changed lines of the file:
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@@
+		)
+	)
+	(wire
+		(pts
+			(xy 177.8 48.26) (xy 166.37 48.26)
+		)
+		(stroke
+			(width 0)
+			(type default)
 		)
 	)
 	(text "Connectors\n-------\nHDMI (type E) port"
 		(exclude_from_sim no)
-		(at 179.832 53.594 0)
+		(at 179.832 57.912 0)
 		(effects
 			(font
@@
 		)
 	)
+	(label "Board_En"
+		(at 76.2 129.54 0)
+		(fields_autoplaced yes)
+		(effects
+			(font
+				(size 1.27 1.27)
+			)
+			(justify left bottom)
+		)
+	)
 	(label "+5V_RAIL"
 		(at 60.96 43.18 180)
@@
 	(label "+5V_RAIL"
 		(at 166.37 31.75 0)
+		(fields_autoplaced yes)
+		(effects
+			(font
+				(size 1.27 1.27)
+			)
+			(justify left bottom)
+		)
+	)
+	(label "Board_En"
+		(at 166.37 48.26 0)
 		(fields_autoplaced yes)
 		(effects
@@
 	(sheet
 		(at 177.8 29.21)
-		(size 24.13 26.67)
+		(size 24.13 31.75)
 		(fields_autoplaced yes)
 		(stroke
@@
 		)
 		(property "Sheetfile" "HDMI.kicad_sch"
-			(at 177.8 56.4646 0)
+			(at 177.8 61.5446 0)
 			(effects
 				(font
@@
 			(effects
 				(font
+					(size 1.27 1.27)
+				)
+				(justify left)
+			)
+		)
+		(pin "GLOBAL_EN" input
+			(at 177.8 48.26 180)
+			(effects
+				(font
