File: PiBoard.kicad_sch (KiCad schematic)
At the start: 4 parts

Commit message: wow everything could not be worse
Other:
- note added: "Connectors ------- HDMI (type D) port USB C 3.0 (HUB) USB C 2.0 (DBG) USB C 2.0 (PWR)"
- note removed: "Connectors ------- HDMI (type E) port USB C 3.0 (HUB) USB C 2.0 (DBG) USB C 2.0 (PWR)"
Changed lines of the file:
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@@
 	(generator_version "9.0")
 	(paper "A4")
-	(text "Connectors\n-------\nHDMI (type E) port\nUSB C 3.0 (HUB)\nUSB C 2.0 (DBG)\nUSB C 2.0 (PWR)"
+	(text "Connectors\n-------\nHDMI (type D) port\nUSB C 3.0 (HUB)\nUSB C 2.0 (DBG)\nUSB C 2.0 (PWR)"
 		(exclude_from_sim no)
 		(at 88.646 111.76 0)

Commit message: chang
Parts:
- H1, H2, H3, H4: footprint MountingHole:MountingHole_3mm -> MountingHole:MountingHole_3.2mm_M3
Other:
- note added: "Connectors ------- HDMI port USB A 3.0 (HUB) USB C 2.0 (DBG)"
- note removed: "Connectors ------- HDMI (type D) port USB C 3.0 (HUB) USB C 2.0 (DBG) USB C 2.0 (PWR)"
Changed lines of the file:
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@@
 	(generator_version "9.0")
 	(paper "A4")
-	(text "Connectors\n-------\nHDMI (type D) port\nUSB C 3.0 (HUB)\nUSB C 2.0 (DBG)\nUSB C 2.0 (PWR)"
-		(exclude_from_sim no)
-		(at 88.646 111.76 0)
+	(text "Connectors\n-------\nHDMI port\nUSB A 3.0 (HUB)\nUSB C 2.0 (DBG)"
+		(exclude_from_sim no)
+		(at 89.154 110.236 0)
 		(effects
 			(font
@@
 			)
 		)
-		(property "Footprint" "MountingHole:MountingHole_3mm"
+		(property "Footprint" "MountingHole:MountingHole_3.2mm_M3"
 			(at 215.9 102.87 0)
 			(effects
@@
 			)
 		)
-		(property "Footprint" "MountingHole:MountingHole_3mm"
+		(property "Footprint" "MountingHole:MountingHole_3.2mm_M3"
 			(at 215.9 121.92 0)
 			(effects
@@
 			)
 		)
-		(property "Footprint" "MountingHole:MountingHole_3mm"
+		(property "Footprint" "MountingHole:MountingHole_3.2mm_M3"
 			(at 215.9 109.22 0)
 			(effects
@@
 			)
 		)
-		(property "Footprint" "MountingHole:MountingHole_3mm"
+		(property "Footprint" "MountingHole:MountingHole_3.2mm_M3"
 			(at 215.9 115.57 0)
 			(effects

Commit message: jlc shit
Parts:
- H1, H2, H3, H4: JLC (none) -> N/A
Changed lines of the file:
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@@
+			)
+		)
+		(property "JLC" "N/A"
+			(at 215.9 102.87 0)
+			(effects
+				(font
+					(size 1.27 1.27)
+				)
+				(hide yes)
 			)
 		)
@@
 			)
 		)
+		(property "JLC" "N/A"
+			(at 215.9 121.92 0)
+			(effects
+				(font
+					(size 1.27 1.27)
+				)
+				(hide yes)
+			)
+		)
 		(instances
 			(project "PiBoard"
@@
 		)
 		(property "Data" ""
+			(at 215.9 109.22 0)
+			(effects
+				(font
+					(size 1.27 1.27)
+				)
+				(hide yes)
+			)
+		)
+		(property "JLC" "N/A"
 			(at 215.9 109.22 0)
 			(effects
@@
 			(at 215.9 115.57 0)
 			(effects
+				(font
+					(size 1.27 1.27)
+				)
+				(hide yes)
+			)
+		)
+		(property "JLC" "N/A"
+			(at 215.9 115.57 0)
+			(effects
