File: RTC.kicad_sch (KiCad schematic)
At the start: 12 parts, among them J7 Molex 470531000, U1 PCF8563T, U10 EMC2301-1-ACZL-TR, U11 74LVC1G07SE-7, Y2 X32K768S301

Commit message: think im done with schematic
Parts:
- removed U11: 74LVC1G07SE-7, Package_TO_SOT_SMD:SOT-353_SC-70-5, symbol CM4IO:74LVC1G07_copy
- added IC7: 74LVC1G07QSE-7, SOT65P210X110-5N, symbol 74LVC1G07QSE-7:74LVC1G07QSE-7
Connections:
- net +5V_PWR: now also IC7.5 (VCC)
- net GLOBAL_EN: now also IC7.4
- net GND: now also IC7.3 (GND)
- net at C23.1, R18.1: now also IC7.2 (A)
Other:
- note added: "RTC alarms can be used to wake up the CM4 when off or shutdown. If CM4 is already awake when alarm triggers, CM4 is reset. This can be used as watchdog reset"
- note removed: "RTC alarms can be used to wake up the Compute module NB an Alarm triggering while already awake will cause a reset This can be used as a watchdog reset"
- moved on the sheet: C23, R17, R18
