File: USB_Ports_Pwr.kicad_sch (KiCad schematic)
At the start: 20 parts, among them IC10 TPS2553QDBVRQ1, IC2 TPS2553QDBVRQ1, IC3 TPS2553QDBVRQ1, IC9 TPS2553QDBVRQ1

Commit message: fixed erc and removed old schematics
Parts:
- IC10, IC2, IC3, IC9: Arrow Part Number (none) -> TPS2553QDBVRQ1; Arrow Price/Stock (none) -> https://www.arrow.com/en/products/tps2553qdbvrq1/texas-inst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; Height (none) -> 1.45; Manufacturer_Name (none) -> Texas Instruments; Manufacturer_Part_Number (none) -> TPS2553QDBVRQ1; Mouser Part Number (none) -> 595-TPS2553QDBVRQ1; Mouser Price/Stock (none) -> https://www.mouser.co.uk/ProductDetail/Texas-Instruments/TP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
