File: PiBoard.kicad_pcb (KiCad board)
At the start: 4 copper layers, 90.1 x 92.5 mm, 143 parts, among them IC1 TCAN337DCNR, IC2 TPS2553QDBVRQ1, IC3 LM74502HDDFR, IC4 AP64501QSP-13, IC5 74LVC1G07QSE-7, IC6 TPS2553QDBVRQ1, IC7 TPS2553QDBVRQ1, J1 CarLVPowerConnector, J12 RTC Battery Port, J2 Display Breakout, J3 2222, J4 USB_C_Receptacle_USB2.0_16P, J5 USB_C_Receptacle_USB2.0_16P, J6 CarCANConnector, J7 Molex 470531000, J8 CarCANConnector, J9 HDMI_E, Q1 PSMN8R5-40MSDX, SW1 SW_Push, SW2 SW_Push, SW3 SW_Push, U1 RTC PCF8563T, U10 Fan PWM Controller, U13 CDSOT23-T24CAN, U14 MCP2515-E/STVAO, U3 FSUSB42MUX, Y4 8 MHz, Y6 ECS-.327-6

Commit message: my life is horrible
Routing:
- net GND: track 168.5 -> 124.9 mm, vias 73 -> 82
- net +3.3V: track 79.0 -> 77.6 mm
- net /Power Distribution/LV+: vias 3 -> 5
- added copper zone on F.Cu, net GND

Commit message: Schem done? [plz full review], redoing layout
Parts:
- removed C17, C20, C21, C3, C30, C31, C43, C51: 100n, Capacitor_SMD:C_0603_1608Metric
- removed D18: ESD204DQAR, Controls_Pi:ESD204DQAR
- removed IC6: TPS2553QDBVRQ1, Controls_Pi:SOT95P280X145-6N
- removed J12: RTC Battery Port, Controls_Pi:CONN02_530470210_MOL
- removed J4: USB_C_Receptacle_USB2.0_16P, Connector_USB:USB_C_Receptacle_GCT_USB4105-xx-A_16P_TopMnt_Horizontal
- removed Module1: ComputeModule4-CM4, CM4IO:Raspberry-Pi-4-Compute-Module
- removed R27: 100n, Resistor_SMD:R_0603_1608Metric
- removed R28: 82k, Resistor_SMD:R_0603_1608Metric
- removed R29: 10k, Resistor_SMD:R_0603_1608Metric
- removed R36: 0, Resistor_SMD:R_0603_1608Metric
- removed R37, R38: 5.1k, Resistor_SMD:R_0603_1608Metric
- removed R39: 100k, Resistor_SMD:R_0603_1608Metric
- removed R40: 56k, Resistor_SMD:R_0603_1608Metric
- removed SW3: SW_Push, Button_Switch_SMD:SW_SPST_B3SL-1002P
- removed U1: RTC PCF8563T, Package_SO:SOIC-8_3.9x4.9mm_P1.27mm
- removed U10: Fan PWM Controller, Package_SO:MSOP-8_3x3mm_P0.65mm
- removed U3: FSUSB42MUX, Package_SO:MSOP-10_3x3mm_P0.5mm
- removed Y6: ECS-.327-6, Controls_Pi:ECS327616RTR
- added C14: 100n, Capacitor_SMD:C_0603_1608Metric, F.Cu at (144.0, 45.2)
- added D17: TPD4E05U06DQAR, Controls_Pi:IC_TPD4E05U06QDQARQ1, F.Cu at (195.4, 140.7)
- added D19: TPD4E05U06DQAR, Controls_Pi:IC_TPD4E05U06QDQARQ1, F.Cu at (220.0, 127.8)
- added F1: 1A, Fuse:Fuse_0805_2012Metric, F.Cu at (196.3, 146.1)
- added FB3: FerriteBead, Inductor_SMD:L_1206_3216Metric, F.Cu at (139.9, 41.8)
- added IC8: TPS2557QDRBTQ1, Controls_Pi:SON65P300X300X100-9N-D, F.Cu at (200.5, 134.8)
- added J10: USB_C_Receptacle, Connector_USB:USB_C_Receptacle_Molex_105450-0101, F.Cu at (226.4, 115.7)
- added J11: RTC Battery Port, Controls_Pi:CONN02_530470210_MOL, F.Cu at (224.4, 45.3)
- added J14: 4x nano-fit, Connector_JST:JST_SH_BM04B-SRSS-TB_1x04-1MP_P1.00mm_Vertical, F.Cu at (208.0, 38.6)
- added Module2: ComputeModule5-CM5, CM5IO:Raspberry-Pi-5-Compute-Module, F.Cu at (114.4, 123.5)
- added R42: 1k, Resistor_SMD:R_0603_1608Metric, F.Cu at (209.5, 56.3)
- added TP5: TestPoint, TestPoint:TestPoint_Pad_2.0x2.0mm, F.Cu at (94.7, 49.2)
- C10: value 120uF -> 100n
- C13, C16: value 1n -> 100n
- C4: value 100n -> 120uF
- D1: value Activity LED -> Activity
- D10, D8: value ESD204DQAR -> TPD4E05U06DQAR; footprint Controls_Pi:ESD204DQAR -> Controls_Pi:IC_TPD4E05U06QDQARQ1
- D11: value VBUS_Debug LED -> TPD4E05U06DQAR; footprint LED_SMD:LED_0603_1608Metric -> Controls_Pi:IC_TPD4E05U06QDQARQ1
- D12: footprint Controls_Pi:DQA_R-PUSON-N10_ -> Controls_Pi:IC_TPD4E05U06QDQARQ1
- D15: value ESD204DQAR -> VBUS_HUB_LED; footprint Controls_Pi:ESD204DQAR -> LED_SMD:LED_0603_1608Metric
- D2: value PI PWR LED -> PI PWR
- D3: value VBUS_Hub LED -> VBUS_PWR_LED
- D5: value 3.3V PWR LED -> 3.3V PWR
- D6: value BAT54C-7-F -> VBUS_PWR_LED; footprint Package_TO_SOT_SMD:SOT-23 -> LED_SMD:LED_0603_1608Metric
- IC2, IC7: value TPS2553QDBVRQ1 -> TPS2557QDRBTQ1; footprint Controls_Pi:SOT95P280X145-6N -> Controls_Pi:SON65P300X300X100-9N-D
- IC5: value 74LVC1G07QSE-7 -> TPS2557QDRBTQ1; footprint Controls_Pi:SOT65P210X110-5N -> Controls_Pi:SON65P300X300X100-9N-D
- J7: value Molex 470531000 -> USB_C_Receptacle_USB2.0_16P; footprint Connector:FanPinHeader_1x04_P2.54mm_Vertical -> UTSVT_Connectors:USB_C_Receptacle_GCT_USB4105-xx-A_16P_TopMnt_Horizontal
- R10: value 56k -> 1.5k
- R11: value 1M -> 20k
- R12: value 1M -> 100k
- R13: value 8k -> 10k
- R16: value 36k -> 5.1k
- R17, R19: value 1k -> 10k
- R18: value 10k -> 5.1k
- R2: value 2.2k -> 700
- R21, R23: value 10k -> 100k
- R22: value 1k -> 1.5k
- R26: value 10k -> 180k
- R3: value 2.2k -> 1.5k
- R4: value 1k -> 10K 1%
- R5: value 100k -> 180k
- R7: value 1.5k -> 56k
- R8: value 1.5k -> 100k
- R9: value 56k -> 120k
- moved R4 135.1 mm to (208.1, 44.0), turned to 0 degrees
- moved R1 124.0 mm to (209.4, 53.8), turned to 0 degrees
- moved D2 122.7 mm to (205.4, 56.4), turned to 0 degrees
- moved D1 122.2 mm to (205.4, 53.8), turned to 0 degrees
- moved TP2 119.7 mm to (199.3, 58.6), turned to 0 degrees
- moved R25 119.6 mm to (209.4, 58.8), turned to 0 degrees
- moved TP1 117.3 mm to (199.3, 54.5)
- moved D5 115.0 mm to (205.4, 59.0), turned to 0 degrees
- moved R21 113.1 mm to (222.3, 77.2), turned to 90 degrees
- moved IC5 112.0 mm to (217.1, 106.7), turned to 90 degrees
- moved R22 97.7 mm to (225.0, 106.6), turned to 90 degrees
- moved R18 94.2 mm to (219.8, 77.2), turned to 90 degrees
- moved C15 78.3 mm to (139.0, 39.8)
- moved R11 75.7 mm to (138.7, 46.1), turned to 90 degrees
- moved R23 71.4 mm to (205.1, 139.2), turned to 0 degrees
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Connections:
- net /CM4 GPIO/CAN_INTR renamed /CM5 GPIO/CAN_INTR
- net /CM4 GPIO/CAN_SPI_CLK renamed /CM5 GPIO/CAN_SPI_CLK
- net /CM4 GPIO/CAN_SPI_CS renamed /CM5 GPIO/CAN_SPI_CS
- net /CM4 GPIO/CAN_SPI_MISO renamed /CM5 GPIO/CAN_SPI_MISO
- net /CM4 GPIO/CAN_SPI_MOSI renamed /CM5 GPIO/CAN_SPI_MOSI
- net /CM4 GPIO/GPIO13 renamed /CM5 GPIO/GPIO13
- net /CM4 GPIO/GPIO19 renamed /CM5 GPIO/GPIO19
- net /CM4 GPIO/GPIO26 renamed /CM5 GPIO/GPIO26
- net /HDMI and High Speed/HDMI_5V renamed /High Speed/HDMI/HDMI_5V
- net Net-(IC1-CANH) renamed /CarCAN/CAN_H
- net Net-(IC1-CANL) renamed /CarCAN/CAN_L
- C1 pad 1: Net-(IC2-EN) -> +5V
- C12 pad 1: Net-(C12-Pad1) -> /High Speed/USB-C/VBUS_HUB
- C13 pad 1: GNDPWR -> +5V
- C15 pad 1: GNDPWR -> Net-(C15-Pad1)
- C16 pad 1: GNDPWR -> +5V
- C2 pad 1: +5V -> Net-(C2-Pad1)
- C22 pad 1: /CM4 GPIO/RUN_PG -> /CM5 GPIO/PWR_BUTT
- C23 pad 1: /Board_En -> /CM5 GPIO/GLOBAL_EN
- D10 pad 1: /HDMI and High Speed/HDMI0_CK_P -> /High Speed/HDMI0_D2_P
- D10 pad 10: /HDMI and High Speed/HDMI0_CK_PRT_P -> /High Speed/HDMI0_D2_P
- D10 pad 2: /HDMI and High Speed/HDMI0_CK_N -> /High Speed/HDMI0_D2_N
- D10 pad 4: /HDMI and High Speed/HDMI0_D1_P -> /High Speed/HDMI0_D0_P
- D10 pad 5: /HDMI and High Speed/HDMI0_D1_N -> /High Speed/HDMI0_D0_N
- D10 pad 6: /HDMI and High Speed/HDMI0_D1_PRT_N -> /High Speed/HDMI0_D0_N
- D10 pad 7: /HDMI and High Speed/HDMI0_D1_PRT_P -> /High Speed/HDMI0_D0_P
- D10 pad 9: /HDMI and High Speed/HDMI0_CK_PRT_N -> /High Speed/HDMI0_D2_N
- D11 pad 1: GND -> /High Speed/HDMI0_CK_P
- D11 pad 2: Net-(D11-A) -> /High Speed/HDMI0_CK_N
- D12 pad 1: /HDMI and High Speed/HDMI0_CEC -> /High Speed/USB_HUB_D-
- D12 pad 10: /HDMI and High Speed/HDMI0_CEC_PRT -> /High Speed/USB_HUB_D-
- D12 pad 2: unconnected-(D12-D1--Pad2) -> /High Speed/USB_HUB_D+
- D12 pad 4: /HDMI and High Speed/HDMI0_SCL -> unconnected-(D12-D2+-Pad4)
- D12 pad 5: /HDMI and High Speed/HDMI0_SDA -> unconnected-(D12-D2--Pad5)
- D12 pad 6: /HDMI and High Speed/HDMI0_SCL_PRT -> unconnected-(D12-NC_1-Pad6)
- D12 pad 7: /HDMI and High Speed/HDMI0_SDA_PRT -> unconnected-(D12-NC_2-Pad7)
- D12 pad 9: unconnected-(D12-NC_3-Pad9) -> /High Speed/USB_HUB_D+
- D15 pad 1: /USB2.0 high speed/USB_Debug_P -> GND
- D15 pad 2: /USB2.0 high speed/USB_Debug_N -> Net-(D15-A)
- D5 pad 1: GND -> Net-(D5-K)
- D5 pad 2: Net-(D5-A) -> +3.3V
- D6 pad 1: /RTC and Fan/RED -> GND
- D6 pad 2: +3.3V -> Net-(D6-A)
- D8 pad 1: /HDMI and High Speed/HDMI0_D2_P -> /High Speed/USB_DBG_D-
- D8 pad 10: /HDMI and High Speed/HDMI0_D2_PRT_P -> /High Speed/USB_DBG_D-
- D8 pad 2: /HDMI and High Speed/HDMI0_D2_N -> /High Speed/USB_DBG_D+
- D8 pad 4: /HDMI and High Speed/HDMI0_D0_P -> unconnected-(D8-D2+-Pad4)
- D8 pad 5: /HDMI and High Speed/HDMI0_D0_N -> unconnected-(D8-D2--Pad5)
- D8 pad 6: /HDMI and High Speed/HDMI0_D0_PRT_N -> unconnected-(D8-NC_1-Pad6)
- D8 pad 7: /HDMI and High Speed/HDMI0_D0_PRT_P -> unconnected-(D8-NC_2-Pad7)
- D8 pad 9: /HDMI and High Speed/HDMI0_D2_PRT_N -> /High Speed/USB_DBG_D+
- FB1 pad 1: /USB2.0 high speed/VBUS_Hub -> /High Speed/USB-C/VBUS_DBG
- FB1 pad 2: Net-(C10-Pad1) -> Net-(C2-Pad1)
- FB2 pad 1: /USB2.0 high speed/VBUS_Debug -> Net-(C10-Pad1)
- FB2 pad 2: Net-(C12-Pad1) -> /High Speed/USB-C/VBUS_HUB
- IC2 pad 1: +5V -> GND
- IC2 pad 2: GND -> +5V
- IC2 pad 3: Net-(IC2-EN) -> +5V
- IC2 pad 6: /USB2.0 high speed/VBUS_Hub -> /High Speed/USB-C/VBUS_DBG
- IC5 pad 1: unconnected-(IC5-NC-Pad1) -> GND
- IC5 pad 2: /CM4 GPIO/nPWR_LED -> +5V
- IC5 pad 3: GND -> +5V
- IC5 pad 4: Net-(IC5-Pad4) -> Net-(IC5-EN)
- IC5 pad 5: +3.3V -> Net-(IC5-ILIM)
- IC7 pad 1: /USB2.0 high speed/VBUS_Debug -> GND
- IC7 pad 2: GND -> /High Speed/USB-C/VBUS_PWR
- IC7 pad 3: Net-(IC7-EN) -> /High Speed/USB-C/VBUS_PWR
- J2 pad 1: +24V -> Net-(J2-+24V)
- J3 pad 10: /CM4 GPIO/GPIO15 -> /CM5 GPIO/GPIO15
- J3 pad 11: /CM4 GPIO/GPIO17 -> /CM5 GPIO/GPIO17
- J3 pad 12: /CM4 GPIO/GPIO18 -> /CM5 GPIO/GPIO18
- J3 pad 13: /CM4 GPIO/GPIO27 -> /CM5 GPIO/GPIO27
- J3 pad 15: /CM4 GPIO/GPIO22 -> /CM5 GPIO/GPIO22
- J3 pad 16: /CM4 GPIO/GPIO23 -> /CM5 GPIO/GPIO23
- J3 pad 18: /CM4 GPIO/GPIO24 -> /CM5 GPIO/GPIO24
- J3 pad 22: /CM4 GPIO/GPIO25 -> /CM5 GPIO/GPIO25
- J3 pad 26: /CM4 GPIO/GPIO7 -> /CM5 GPIO/GPIO7
- J3 pad 27: /CM4 GPIO/GPIO0 -> /CM5 GPIO/GPIO0
- J3 pad 28: /CM4 GPIO/GPIO1 -> /CM5 GPIO/GPIO1
- J3 pad 29: /CM4 GPIO/GPIO5 -> /CM5 GPIO/GPIO5
- J3 pad 3: /CM4 GPIO/GPIO2 -> /CM5 GPIO/GPIO2
- J3 pad 31: /CM4 GPIO/GPIO6 -> /CM5 GPIO/GPIO6
- J3 pad 36: /CM4 GPIO/GPIO16 -> /CM5 GPIO/GPIO16
- J3 pad 38: /CM4 GPIO/GPIO20 -> /CM5 GPIO/GPIO20
- J3 pad 40: /CM4 GPIO/GPIO21 -> /CM5 GPIO/GPIO21
- J3 pad 5: /CM4 GPIO/GPIO3 -> /CM5 GPIO/GPIO3
- J3 pad 7: /CM4 GPIO/GPIO4 -> /CM5 GPIO/GPIO4
- J3 pad 8: /CM4 GPIO/GPIO14 -> /CM5 GPIO/GPIO14
- J5 pad A4: Net-(C10-Pad1) -> Net-(C2-Pad1)
- J5 pad A6: /USB2.0 high speed/USB_Hub_PRT_P -> /High Speed/USB_DBG_D+
- J5 pad A7: /USB2.0 high speed/USB_Hub_PRT_N -> /High Speed/USB_DBG_D-
- J5 pad A8: /USB2.0 high speed/SBU1_Hub -> unconnected-(J5-SBU1-PadA8)
- J5 pad A9: Net-(C10-Pad1) -> Net-(C2-Pad1)
- J5 pad B4: Net-(C10-Pad1) -> Net-(C2-Pad1)
- J5 pad B6: /USB2.0 high speed/USB_Hub_PRT_P -> /High Speed/USB_DBG_D+
- J5 pad B7: /USB2.0 high speed/USB_Hub_PRT_N -> /High Speed/USB_DBG_D-
- J5 pad B8: /USB2.0 high speed/SBU2_Hub -> unconnected-(J5-SBU2-PadB8)
- J5 pad B9: Net-(C10-Pad1) -> Net-(C2-Pad1)
- J5 pad S1: GNDPWR -> GND
- J9 pad 1: /HDMI and High Speed/HDMI0_D2_PRT_P -> /High Speed/HDMI0_D2_P
- J9 pad 10: /HDMI and High Speed/HDMI0_CK_PRT_P -> /High Speed/HDMI0_CK_P
- J9 pad 12: /HDMI and High Speed/HDMI0_CK_PRT_N -> /High Speed/HDMI0_CK_N
- J9 pad 13: /HDMI and High Speed/HDMI0_CEC_PRT -> /High Speed/HDMI0_CEC
- J9 pad 15: /HDMI and High Speed/HDMI0_SCL_PRT -> /High Speed/HDMI0_SCL
- J9 pad 16: /HDMI and High Speed/HDMI0_SDA_PRT -> /High Speed/HDMI0_SDA
- J9 pad 19: /HDMI and High Speed/HDMI0_HOTPLUG -> /High Speed/HDMI0_HOTPLUG
- J9 pad 3: /HDMI and High Speed/HDMI0_D2_PRT_N -> /High Speed/HDMI0_D2_N
- J9 pad 4: /HDMI and High Speed/HDMI0_D1_PRT_P -> /High Speed/HDMI0_D1_P
- J9 pad 6: /HDMI and High Speed/HDMI0_D1_PRT_N -> /High Speed/HDMI0_D1_N
- J9 pad 7: /HDMI and High Speed/HDMI0_D0_PRT_P -> /High Speed/HDMI0_D0_P
- J9 pad 9: /HDMI and High Speed/HDMI0_D0_PRT_N -> /High Speed/HDMI0_D0_N
- R1 pad 2: Net-(Module1A-PI_nLED_Activity) -> /CM5 GPIO/LED_nACT
- R10 pad 1: +5V -> /High Speed/USB-C/VBUS_PWR
- R10 pad 2: Net-(J5-CC2) -> Net-(D6-A)
- R11 pad 1: GND -> Net-(IC7-ILIM)
- R11 pad 2: GNDPWR -> GND
- R12 pad 1: GND -> /High Speed/USB-C/VBUS_PWR
- R12 pad 2: GNDPWR -> Net-(IC7-EN)
- R16 pad 1: +3.3V -> GND
- R16 pad 2: Net-(J7-Pin_3) -> Net-(J5-CC1)
- R17 pad 2: /CM4 GPIO/RUN_PG -> /CM5 GPIO/PWR_BUTT
- R18 pad 1: +5V -> GND
- R18 pad 2: /CM4 GPIO/RUN_PG -> Net-(J5-CC2)
- R19 pad 2: /Board_En -> /CM5 GPIO/GLOBAL_EN
- R21 pad 1: +5V -> /CM5 GPIO/GLOBAL_EN
- R21 pad 2: /Board_En -> Net-(IC2-EN)
- R22 pad 1: Net-(R22-Pad1) -> /High Speed/USB-C/VBUS_HUB
- R22 pad 2: /CM4 GPIO/GPIO3 -> Net-(D15-A)
- R23 pad 1: +5V -> /CM5 GPIO/GLOBAL_EN
- R23 pad 2: /CM4 GPIO/GPIO3 -> Net-(IC8-EN)
- R25 pad 1: +3.3V -> Net-(D5-K)
- R25 pad 2: Net-(D5-A) -> GND
- R26 pad 1: +3.3V -> Net-(IC8-ILIM)
- R26 pad 2: /CM4 GPIO/SCL0 -> GND
- R3 pad 1: /HDMI and High Speed/USBOTG_ID -> /High Speed/USB-C/VBUS_DBG
- R3 pad 2: GND -> Net-(D3-A)
- R4 pad 1: Net-(D2-K) -> /CM5 GPIO/FAN_PWM
- R4 pad 2: Net-(IC5-Pad4) -> +3.3V
- R5 pad 1: /Board_En -> Net-(IC2-ILIM)
- R5 pad 2: Net-(IC2-EN) -> GND
- R6 pad 1: GND -> Net-(J10-CC1)
- R6 pad 2: Net-(IC2-ILIM) -> +5V
- R7 pad 1: /USB2.0 high speed/VBUS_Hub -> Net-(J10-CC2)
- R7 pad 2: Net-(D3-A) -> +5V
- R8 pad 1: /USB2.0 high speed/VBUS_Debug -> Net-(IC5-EN)
- R8 pad 2: Net-(D11-A) -> /CM5 GPIO/GLOBAL_EN
- R9 pad 1: +5V -> Net-(IC5-ILIM)
- R9 pad 2: Net-(J5-CC1) -> GND
- S1 pad 2: /CM4 GPIO/BT_Disable -> /CM5 GPIO/BT_Disable
- S1 pad 5: /CM4 GPIO/WiFi_Disable -> /CM5 GPIO/WiFi_Disable
- S2 pad 2: /CM4 GPIO/EEPROM_nWP -> /CM5 GPIO/EEPROM_nWP
- S2 pad 5: /CM4 GPIO/nRPIBOOT -> /CM5 GPIO/nRPIBOOT
- TP1 pad 1: Net-(D1-K) -> +24V
- TP2 pad 1: Net-(D2-K) -> +5V
Routing:
- net /Board_En: track 135.4 -> 0.00 mm, vias 6 -> 0
- net /CM4 GPIO/SDA0: track 105.3 -> 0.00 mm, vias 4 -> 0
- net /CM4 GPIO/SCL0: track 99.3 -> 0.00 mm, vias 4 -> 0
- net /CM4 GPIO/GPIO3: track 84.2 -> 0.00 mm, vias 2 -> 0
- net /CM5 GPIO/GPIO3: track 0.00 -> 79.1 mm, vias 0 -> 2
- net /CM5 GPIO/EEPROM_nWP: track 0.00 -> 77.9 mm, vias 0 -> 3
- net /CM4 GPIO/EEPROM_nWP: track 77.9 -> 0.00 mm, vias 3 -> 0
- net /CM5 GPIO/BT_Disable: track 0.00 -> 73.6 mm, vias 0 -> 3
- net /CM4 GPIO/BT_Disable: track 73.6 -> 0.00 mm, vias 3 -> 0
- net /CM5 GPIO/WiFi_Disable: track 0.00 -> 71.8 mm, vias 0 -> 3
- net /CM4 GPIO/WiFi_Disable: track 71.8 -> 0.00 mm, vias 3 -> 0
- net unconnected-(Module2A-SDA0-Pad82): track 0.00 -> 64.7 mm, vias 0 -> 2
- net /CM5 GPIO/nRPIBOOT: track 0.00 -> 59.2 mm, vias 0 -> 3
- net /CM4 GPIO/nRPIBOOT: track 59.2 -> 0.00 mm, vias 3 -> 0
- net /CM5 GPIO/GPIO22: track 0.00 -> 58.2 mm, vias 0 -> 1
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- removed copper zone on F.Cu, net +5V
- removed copper zone on In2.Cu, net /Power Distribution/LV+
- removed copper zone on In1.Cu, net GND

Commit message: I hate my life
Parts:
- removed C26: 22n, Capacitor_SMD:C_0603_1608Metric
- removed C4: 120uF, Capacitor_SMD:C_0603_1608Metric
- removed J9: HDMI_E, Controls_Pi:MX50019NQ1
- removed Z2: SMAF4751A-TP, UTSVT_Passives:SODFL5026X125N
- added C3: 0.1u, Capacitor_SMD:C_0603_1608Metric_Pad1.08x0.95mm_HandSolder, F.Cu at (106.3, 77.5)
- added J4: HDMI_D_1.4, Connector_Video:HDMI_Micro-D_Molex_46765-1x01, F.Cu at (130.3, 141.4)
- added R27: 10K, Resistor_SMD:R_0603_1608Metric_Pad0.98x0.95mm_HandSolder, F.Cu at (121.3, 95.9)
- C1, C10, C11, C12, C13, C14, C15, C16, C2, C22, C23, C36, C37, C5, C56, C59, C60, C7: footprint Capacitor_SMD:C_0603_1608Metric -> Capacitor_SMD:C_0603_1608Metric_Pad1.08x0.95mm_HandSolder
- C18, C19, C27, C6, C61, C8, C9: footprint Capacitor_SMD:C_0603_1608Metric -> Capacitor_SMD:C_0805_2012Metric_Pad1.18x1.45mm_HandSolder
- C24, C25: value 26 pF -> 22 pF; footprint Capacitor_SMD:C_0603_1608Metric -> Capacitor_SMD:C_0603_1608Metric_Pad1.08x0.95mm_HandSolder
- C29, C58: footprint Capacitor_SMD:C_0805_2012Metric -> Capacitor_SMD:C_0805_2012Metric_Pad1.18x1.45mm_HandSolder
- D1, D13, D14, D15, D16, D2, D3, D4, D5, D6, D7, D9: footprint LED_SMD:LED_0603_1608Metric -> LED_SMD:LED_0603_1608Metric_Pad1.05x0.95mm_HandSolder
- F1: value 1A -> 3568; footprint Fuse:Fuse_0805_2012Metric -> Controls_Pi:FUSE_3568
- Q1: footprint UTSVT_Power_SP:PSMN8R5-40MSDX -> UTSVT_Power:PSMN8R5-40MSDX
- R1, R42: value 1k -> 700; footprint Resistor_SMD:R_0603_1608Metric -> Resistor_SMD:R_0603_1608Metric_Pad0.98x0.95mm_HandSolder
- R10, R100, R11, R12, R13, R14, R15, R16, R17, R18, R19, R2, R20, R21, R22, R23, R24, R25, R26, R3, R33, R34, R35, R44, R45, R5, R6, R7, R8, R9: footprint Resistor_SMD:R_0603_1608Metric -> Resistor_SMD:R_0603_1608Metric_Pad0.98x0.95mm_HandSolder
- R30, R31: footprint Resistor_SMD:R_0805_2012Metric -> Resistor_SMD:R_0805_2012Metric_Pad1.20x1.40mm_HandSolder
- R4: value 10K 1% -> 10K; footprint Resistor_SMD:R_0603_1608Metric -> Resistor_SMD:R_0603_1608Metric_Pad0.98x0.95mm_HandSolder
- moved R1 143.7 mm to (70.1, 89.0), turned to -90 degrees
- moved R42 141.6 mm to (71.8, 89.0), turned to -90 degrees
- moved R25 139.3 mm to (73.5, 89.0), turned to -90 degrees
- moved D1 139.0 mm to (70.1, 85.5), turned to 90 degrees
- moved D2 136.8 mm to (71.8, 85.5), turned to 90 degrees
- moved D5 134.6 mm to (73.5, 85.5), turned to 90 degrees
- moved TP2 133.5 mm to (66.2, 69.4)
- moved F1 124.6 mm to (93.6, 75.6), turned to -90 degrees
- moved R21 112.1 mm to (116.9, 115.5), turned to 0 degrees
- moved D9 111.3 mm to (91.8, 84.8), turned to 0 degrees
- moved R44 109.8 mm to (95.2, 84.8), turned to 180 degrees
- moved J11 109.1 mm to (126.6, 93.5)
- moved TP5 109.1 mm to (114.1, 156.5)
- moved R4 108.2 mm to (113.2, 95.9), turned to 180 degrees
- moved J14 106.1 mm to (117.3, 93.6)
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Connections:
- D11 pad 1: /High Speed/HDMI0_CK_P -> /High Speed/HDMI0_CK_N
- D11 pad 10: /High Speed/HDMI0_CK_P -> /High Speed/HDMI0_CK_N
- D11 pad 2: /High Speed/HDMI0_CK_N -> /High Speed/HDMI0_CK_P
- D11 pad 4: /High Speed/HDMI0_D1_P -> /High Speed/HDMI0_D1_N
- D11 pad 5: /High Speed/HDMI0_D1_N -> /High Speed/HDMI0_D1_P
- D11 pad 6: /High Speed/HDMI0_D1_N -> /High Speed/HDMI0_D1_P
- D11 pad 7: /High Speed/HDMI0_D1_P -> /High Speed/HDMI0_D1_N
- D11 pad 9: /High Speed/HDMI0_CK_N -> /High Speed/HDMI0_CK_P
- D12 pad 1: /High Speed/USB_HUB_D- -> unconnected-(D12-D1+-Pad1)
- D12 pad 10: /High Speed/USB_HUB_D- -> unconnected-(D12-NC_4-Pad10)
- D12 pad 2: /High Speed/USB_HUB_D+ -> unconnected-(D12-D1--Pad2)
- D12 pad 4: unconnected-(D12-D2+-Pad4) -> /High Speed/USB_HUB_D-
- D12 pad 5: unconnected-(D12-D2--Pad5) -> /High Speed/USB_HUB_D+
- D12 pad 6: unconnected-(D12-NC_1-Pad6) -> /High Speed/USB_HUB_D+
- D12 pad 7: unconnected-(D12-NC_2-Pad7) -> /High Speed/USB_HUB_D-
- D12 pad 9: /High Speed/USB_HUB_D+ -> unconnected-(D12-NC_3-Pad9)
- D17 pad 2: /High Speed/HDMI0_HOTPLUG -> /High Speed/HDMI0_SCL
- D17 pad 4: /High Speed/HDMI0_SCL -> /High Speed/HDMI0_SDA
- D17 pad 5: /High Speed/HDMI0_SDA -> /High Speed/HDMI0_HOTPLUG
- D17 pad 6: /High Speed/HDMI0_SDA -> /High Speed/HDMI0_HOTPLUG
- D17 pad 7: /High Speed/HDMI0_SCL -> /High Speed/HDMI0_SDA
- D17 pad 9: /High Speed/HDMI0_HOTPLUG -> /High Speed/HDMI0_SCL
- D8 pad 1: /High Speed/USB_DBG_D- -> unconnected-(D8-D1+-Pad1)
- D8 pad 10: /High Speed/USB_DBG_D- -> unconnected-(D8-NC_4-Pad10)
- D8 pad 2: /High Speed/USB_DBG_D+ -> unconnected-(D8-D1--Pad2)
- D8 pad 4: unconnected-(D8-D2+-Pad4) -> /High Speed/USB_DBG_D-
- D8 pad 5: unconnected-(D8-D2--Pad5) -> /High Speed/USB_DBG_D+
- D8 pad 6: unconnected-(D8-NC_1-Pad6) -> /High Speed/USB_DBG_D+
- D8 pad 7: unconnected-(D8-NC_2-Pad7) -> /High Speed/USB_DBG_D-
- D8 pad 9: /High Speed/USB_DBG_D+ -> unconnected-(D8-NC_3-Pad9)
- Q1 pad 1: /Power Distribution/LV+ -> +24V
- Q1 pad 10: +24V -> /Power Distribution/LV+
- Q1 pad 11: +24V -> /Power Distribution/LV+
- Q1 pad 2: /Power Distribution/LV+ -> +24V
- Q1 pad 3: /Power Distribution/LV+ -> +24V
- Q1 pad 5: +24V -> /Power Distribution/LV+
- Q1 pad 6: +24V -> /Power Distribution/LV+
- Q1 pad 7: +24V -> /Power Distribution/LV+
- Q1 pad 8: +24V -> /Power Distribution/LV+
- Q1 pad 9: +24V -> /Power Distribution/LV+
Routing:
- net /CM5 GPIO/EEPROM_nWP: track 77.9 -> 8.60 mm, vias 3 -> 1
- net /CM5 GPIO/BT_Disable: track 73.6 -> 11.6 mm, vias 3 -> 1
- net /CM5 GPIO/WiFi_Disable: track 71.8 -> 11.4 mm, vias 3 -> 1
- net /CM5 GPIO/nRPIBOOT: track 59.2 -> 11.8 mm, vias 3 -> 1
- net /CM5 GPIO/GPIO13: track 91.1 -> 50.0 mm, vias 5 -> 3
- net /CM5 GPIO/GPIO19: track 87.5 -> 46.6 mm, vias 5 -> 3
- net /CM5 GPIO/GPIO26: track 84.3 -> 43.6 mm, vias 5 -> 3
- net unconnected-(Module2A-SDA0-Pad82): track 64.7 -> 29.1 mm
- net /CM5 GPIO/PWR_BUTT: track 47.1 -> 12.9 mm, vias 4 -> 3
- net +5V: track 47.0 -> 17.6 mm, vias 1 -> 0
- net /CM5 GPIO/GPIO3: track 79.1 -> 51.3 mm, vias 2 -> 1
- net unconnected-(Module2A-SCL0-Pad80): track 0.00 -> 24.8 mm, vias 0 -> 2
- net +3.3V: track 39.2 -> 19.6 mm, vias 2 -> 0
- net /CM5 GPIO/CAN_SPI_CS: track 43.5 -> 26.1 mm
- net +1.8V: track 26.8 -> 9.40 mm
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- added copper zone on F.Cu, net +5V
- added copper zone on F.Cu, net /High Speed/USB-C/VBUS_DBG
- added copper zone on F.Cu, net /High Speed/USB-C/VBUS_HUB
- added copper zone on F.Cu, net /High Speed/USB-C/VBUS_PWR
- added copper zone on F.Cu, net Net-(C15-Pad1)
- added copper zone on F.Cu, net Net-(C2-Pad1)
- added copper zone on F.Cu, net Net-(IC4-SW)
- added copper zone on F.Cu, net Net-(J2-+24V)
- removed copper zone on F.Cu, net +3.3V
- removed copper zone on B.Cu, net GND
Other:
- board text added: "For Instructional Use Only."
- board text added: "SOLIDWORKS Educational Product."
- board text removed: "Left some of these pwr components 0805 (?)"
- board text removed: "Trying to keep this space more open for fancy routing ig"

Commit message: I'm unhappy with the state of the world
Parts:
- J10: footprint Connector_USB:USB_C_Receptacle_Molex_105450-0101 -> Controls_Pi:CONN_221608-0001_MOL
- J5: footprint Connector_USB:USB_C_Receptacle_GCT_USB4105-xx-A_16P_TopMnt_Horizontal -> Controls_Pi:2193200001
- J7: footprint UTSVT_Connectors:USB_C_Receptacle_GCT_USB4105-xx-A_16P_TopMnt_Horizontal -> Controls_Pi:2193200001
- moved C14 43.7 mm to (119.7, 148.9)
- moved R11 43.7 mm to (118.7, 142.8)
- moved R12 43.7 mm to (120.2, 142.8)
- moved FB3 43.7 mm to (123.9, 144.8)
- moved IC7 43.7 mm to (120.1, 146.3)
- moved J7 42.6 mm to (129.2, 144.5)
- moved D6 42.6 mm to (129.5, 150.7)
- moved R10 42.6 mm to (126.2, 150.7)
- moved C15 36.4 mm to (123.8, 141.7), turned to 180 degrees
- moved H1 33.9 mm to (85.6, 89.1)
- moved H4 17.5 mm to (121.0, 155.4)
- moved R16 16.9 mm to (133.9, 107.4), turned to 90 degrees
- moved R6 16.1 mm to (132.9, 121.8), turned to -90 degrees
- moved D12 14.0 mm to (133.1, 118.4), turned to 180 degrees
- moved D11 12.8 mm to (118.9, 129.0)
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Connections:
- D8 pad 1: unconnected-(D8-D1+-Pad1) -> /High Speed/USB_DBG_D-
- D8 pad 10: unconnected-(D8-NC_4-Pad10) -> /High Speed/USB_DBG_D-
- D8 pad 2: unconnected-(D8-D1--Pad2) -> /High Speed/USB_DBG_D+
- D8 pad 4: /High Speed/USB_DBG_D- -> unconnected-(D8-D2+-Pad4)
- D8 pad 5: /High Speed/USB_DBG_D+ -> unconnected-(D8-D2--Pad5)
- D8 pad 6: /High Speed/USB_DBG_D+ -> unconnected-(D8-NC_1-Pad6)
- D8 pad 7: /High Speed/USB_DBG_D- -> unconnected-(D8-NC_2-Pad7)
- D8 pad 9: unconnected-(D8-NC_3-Pad9) -> /High Speed/USB_DBG_D+
Routing:
- net GND: track 152.4 -> 118.8 mm
- net Net-(J5-CC2): track 6.86 -> 0.00 mm, vias 2 -> 0
- net Net-(J5-CC1): track 6.68 -> 0.00 mm, vias 2 -> 0
- net /High Speed/USB-C/VBUS_PWR: track 13.1 -> 6.44 mm
- removed copper zone on F.Cu, net Net-(C2-Pad1)
Other:
- board size 90.1 x 92.5 mm -> 81 x 92.4 mm
- board text added: "Fuckass constraints"
- board text added: "I mean what am I supposed to do here"

Commit message: rrr
Parts:
- moved H2 12.9 mm to (130.1, 94.9)
- moved J11 3.94 mm to (123.3, 92.6)
Routing:
- net GND: track 118.8 -> 116.1 mm
Other:
- board size 81 x 92.4 mm -> 74.2 x 92.4 mm
Changed lines of the file:
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@@
 	(footprint "Controls_Pi:CONN02_530470210_MOL"
 		(layer "F.Cu")
-		(at 126.95 94.2 180)
+		(at 123.35 92.6 180)
 		(tags "530470210 ")
 		(property "Reference" "J11"
@@
 	(footprint "MountingHole:MountingHole_3mm"
 		(layer "F.Cu")
-		(at 135.2 83)
+		(at 130.1 94.9)
 		(descr "Mounting Hole 3mm, no annular, generated by kicad-footprint-generator mountinghole.py")
 		(tags "mountinghole")
@@
 	)
 	(gr_line
-		(start 142.7525 94.4)
+		(start 136 94.1)
 		(end 134 66.761966)
 		(stroke
@@
 	(gr_line
 		(start 123.68 159.2)
-		(end 142.7525 144.6)
+		(end 136 148.7)
 		(stroke
 			(width 0.05)
@@
 	)
 	(gr_line
-		(start 142.7525 94.4)
-		(end 142.7525 144.6)
+		(start 136 94.1)
+		(end 136 148.7)
 		(stroke
 			(width 0.05)
@@
 	)
 	(segment
-		(start 202.5375 73.8)
-		(end 202.5375 72.4125)
-		(width 0.25)
-		(layer "F.Cu")
-		(net 2)
-	)
-	(segment
 		(start 123.4775 86.163501)
 		(end 123.4775 86.176)
@@
 		(width 0.15)
 		(layer "F.Cu")
-		(net 2)
-	)
-	(segment
-		(start 167.1 30.805)
-		(end 168.42528 30.805)
-		(width 0.15)
-		(layer "F.Cu")

Commit message: frank
Parts:
- removed Q1: PSMN8R5-40MSDX, UTSVT_Power:PSMN8R5-40MSDX
- added Q2: NVMFWS1D7N04XMT1G, Controls_Pi:NVMFWS3D0P04M8LT1G, F.Cu at (109.5, 82.1)
- added Q3: NVMFWS1D7N04XMT1G, Controls_Pi:NVMFWS3D0P04M8LT1G, F.Cu at (101.0, 82.1)
- moved D16 44.3 mm to (108.9, 67.5), turned to 0 degrees
- moved R33 42.8 mm to (105.4, 67.5), turned to 180 degrees
- moved D1 42.1 mm to (108.9, 69.2), turned to 0 degrees
- moved R1 40.5 mm to (105.4, 69.2), turned to 180 degrees
- moved D2 31.7 mm to (97.9, 67.5), turned to 0 degrees
- moved R42 31.2 mm to (94.4, 67.5), turned to 180 degrees
- moved H1 29.5 mm to (66.3, 66.8)
- moved D5 29.3 mm to (97.9, 69.2), turned to 0 degrees
- moved R25 28.8 mm to (94.4, 69.2), turned to 180 degrees
- moved H2 27.9 mm to (128.2, 67.1)
- moved R20 27.7 mm to (82.5, 67.5), turned to 180 degrees
- moved D14 27.7 mm to (86.0, 67.5), turned to 0 degrees
- moved R15 25.3 mm to (82.5, 69.2), turned to 180 degrees
- moved D13 25.3 mm to (86.0, 69.2), turned to 0 degrees
- moved TP1 12.4 mm to (87.1, 86.0)
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Connections:
- J14 pad 1: +24V -> +5V
- Z1 pad 1: /Power Distribution/RPP_EN -> /Power Distribution/LV+
Routing:
- net /CM5 GPIO/GLOBAL_EN: track 14.1 -> 103.3 mm, vias 1 -> 4
- net /CM5 GPIO/CAN_SPI_MISO: track 68.6 -> 121.8 mm, vias 1 -> 2
- net /CM5 GPIO/CAN_SPI_MOSI: track 81.6 -> 133.9 mm, vias 1 -> 2
- net /CM5 GPIO/CAN_SPI_CS: track 26.1 -> 78.1 mm, vias 3 -> 4
- net /CM5 GPIO/CAN_SPI_CLK: track 82.3 -> 132.4 mm, vias 3 -> 4
- net /CM5 GPIO/EEPROM_nWP: track 8.60 -> 57.6 mm, vias 1 -> 3
- net /CM5 GPIO/CAN_INTR: track 26.0 -> 74.0 mm, vias 2 -> 3
- net /CM5 GPIO/BT_Disable: track 11.6 -> 53.4 mm, vias 1 -> 2
- net /CM5 GPIO/WiFi_Disable: track 11.4 -> 51.4 mm, vias 1 -> 2
- net GND: track 116.1 -> 153.4 mm, vias 6 -> 19
- net /CM5 GPIO/LED_nACT: track 36.1 -> 2.19 mm
- net /CM5 GPIO/nRPIBOOT: track 11.8 -> 39.9 mm, vias 1 -> 2
- net /CM5 GPIO/nPWR_LED: track 18.6 -> 0.00 mm
- net /CM5 GPIO/PWR_BUTT: track 12.9 -> 31.3 mm, vias 3 -> 4
- net /High Speed/HDMI/HDMI_5V: track 0.00 -> 8.84 mm
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- added copper zone on F.Cu, net /High Speed/HDMI/HDMI_5V
- added copper zone on F.Cu, net Net-(C2-Pad1)
- added copper zone on F.Cu, net Net-(Q2-Pad1)
Other:
- board size 74.2 x 92.4 mm -> 74.2 x 101.4 mm

Commit message: frank2
Parts:
- removed R12, R21, R23, R8: 100k, Resistor_SMD:R_0603_1608Metric_Pad0.98x0.95mm_HandSolder
- moved R25 88.6 mm to (58.4, 150.2), turned to -90 degrees
- moved D5 86.9 mm to (58.4, 146.7), turned to 90 degrees
- moved TP5 79.4 mm to (115.7, 77.2)
- moved J11 78.2 mm to (66.9, 149.2)
- moved R42 74.2 mm to (58.0, 132.2), turned to -90 degrees
- moved D2 73.0 mm to (58.0, 128.7), turned to 90 degrees
- moved D1 66.2 mm to (58.9, 112.7), turned to 90 degrees
- moved R1 66.1 mm to (58.9, 116.2), turned to -90 degrees
- moved D16 55.8 mm to (58.6, 91.8), turned to 90 degrees
- moved R33 54.4 mm to (58.6, 95.3), turned to -90 degrees
- moved D13 42.1 mm to (50.3, 91.6), turned to 90 degrees
- moved R15 41.3 mm to (50.3, 95.1), turned to -90 degrees
- moved D14 39.6 mm to (54.6, 91.7), turned to 90 degrees
- moved R20 39.3 mm to (54.6, 95.1), turned to -90 degrees
- moved R27 10.3 mm to (111.0, 101.3), turned to -90 degrees
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Connections:
- IC2 pad 4: Net-(IC2-EN) -> /CM5 GPIO/GLOBAL_EN
- IC5 pad 4: Net-(IC5-EN) -> /CM5 GPIO/GLOBAL_EN
- IC7 pad 4: Net-(IC7-EN) -> /High Speed/USB-C/VBUS_PWR
- IC8 pad 4: Net-(IC8-EN) -> /CM5 GPIO/GLOBAL_EN
Routing:
- net +3.3V: track 11.1 -> 167.4 mm, vias 0 -> 6
- net /CM5 GPIO/CC2: track 0.00 -> 77.8 mm, vias 0 -> 2
- net /CM5 GPIO/CC1: track 0.00 -> 66.3 mm, vias 0 -> 2
- net /CM5 GPIO/FAN_PWM: track 0.00 -> 55.2 mm, vias 0 -> 4
- net /CM5 GPIO/FAN_TACHO: track 0.00 -> 46.8 mm, vias 0 -> 2
- net GND: track 153.4 -> 195.2 mm, vias 19 -> 54
- net unconnected-(Module2A-SDA0-Pad82): track 29.1 -> 0.00 mm, vias 2 -> 0
- net /CM5 GPIO/RTC_Batt: track 0.00 -> 28.8 mm, vias 0 -> 1
- net unconnected-(Module2A-SCL0-Pad80): track 24.8 -> 0.00 mm, vias 2 -> 0
- net /CM5 GPIO/GLOBAL_EN: track 103.3 -> 110.1 mm
- net +5V: track 17.6 -> 22.4 mm
- net Net-(IC2-EN): track 2.65 -> 0.00 mm
- net Net-(IC7-EN): track 2.53 -> 0.00 mm
- net Net-(IC8-EN): track 1.94 -> 0.00 mm
- net Net-(IC5-EN): track 1.88 -> 0.00 mm
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- added copper zone on F.Cu, net +3.3V
- added copper zone on B.Cu, net GND
Other:
- board size 74.2 x 101.4 mm -> 71.5 x 97.1 mm

Commit message: Copy of I hate my life pt2.5 final final (3)
Parts:
- moved R25 99.5 mm to (115.8, 68.9), turned to 180 degrees
- moved D5 98.8 mm to (119.3, 68.9), turned to 0 degrees
- moved D13 54.4 mm to (99.7, 68.9), turned to 0 degrees
- moved R15 52.8 mm to (96.2, 68.9), turned to 180 degrees
- moved R42 45.4 mm to (69.6, 88.2), turned to 0 degrees
- moved D2 41.2 mm to (66.1, 88.2), turned to 180 degrees
- moved D14 40.5 mm to (88.0, 68.8), turned to 0 degrees
- moved R20 39.9 mm to (84.6, 68.8), turned to 180 degrees
- moved R33 30.0 mm to (72.7, 68.8), turned to 180 degrees
- moved D16 28.9 mm to (76.2, 68.8), turned to 0 degrees
- moved R1 27.2 mm to (69.5, 91.2), turned to 0 degrees
- moved D1 22.7 mm to (66.1, 91.2), turned to 180 degrees
- moved D8 2.04 mm to (120.3, 110.7)
- moved D10 1.90 mm to (114.8, 127.2)
- moved D11 1.90 mm to (114.8, 130.2)
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Connections:
- D10 pad 4: /High Speed/HDMI0_D0_P -> /High Speed/HDMI0_D1_P
- D10 pad 5: /High Speed/HDMI0_D0_N -> /High Speed/HDMI0_D1_N
- D10 pad 6: /High Speed/HDMI0_D0_N -> /High Speed/HDMI0_D1_N
- D10 pad 7: /High Speed/HDMI0_D0_P -> /High Speed/HDMI0_D1_P
- D11 pad 4: /High Speed/HDMI0_D1_N -> /High Speed/HDMI0_D0_N
- D11 pad 5: /High Speed/HDMI0_D1_P -> /High Speed/HDMI0_D0_P
- D11 pad 6: /High Speed/HDMI0_D1_P -> /High Speed/HDMI0_D0_P
- D11 pad 7: /High Speed/HDMI0_D1_N -> /High Speed/HDMI0_D0_N
- IC8 pad 3: unconnected-(IC8-IN_2-Pad3) -> +5V
- IC8 pad 7: unconnected-(IC8-OUT_2-Pad7) -> /High Speed/HDMI/HDMI_5V
- R15 pad 2: /CM5 GPIO/GPIO19 -> /CM5 GPIO/GPIO26
- R20 pad 2: /CM5 GPIO/GPIO13 -> /CM5 GPIO/GPIO19
- R33 pad 2: /CM5 GPIO/GPIO26 -> /CM5 GPIO/GPIO13
Routing:
- net +3.3V: track 167.4 -> 252.1 mm, vias 6 -> 8
- net /CM5 GPIO/GPIO26: track 42.9 -> 90.7 mm, vias 3 -> 4
- net /CM5 GPIO/nPWR_LED: track 0.00 -> 47.0 mm, vias 0 -> 3
- net /CM5 GPIO/GPIO13: track 49.3 -> 91.9 mm, vias 3 -> 4
- net /CM5 GPIO/GPIO19: track 45.8 -> 88.2 mm, vias 3 -> 4
- net /High Speed/HDMI0_HOTPLUG: track 0.00 -> 28.3 mm, vias 0 -> 4
- net /CM5 GPIO/LED_nACT: track 1.50 -> 29.3 mm, vias 1 -> 2
- net /High Speed/USB_DBG_D+: track 0.00 -> 25.2 mm, vias 0 -> 2
- net /High Speed/USB_DBG_D-: track 0.00 -> 25.2 mm, vias 0 -> 2
- net /High Speed/USB_HUB_D+: track 0.00 -> 23.9 mm, vias 0 -> 4
- net /High Speed/USB_HUB_D-: track 0.00 -> 23.9 mm, vias 0 -> 4
- net /High Speed/HDMI0_CEC: track 0.00 -> 22.3 mm, vias 0 -> 2
- net /High Speed/USB_HUB_RX1-: track 0.00 -> 22.1 mm, vias 0 -> 4
- net /High Speed/USB_HUB_RX1+: track 0.00 -> 22.1 mm, vias 0 -> 4
- net /High Speed/USB_HUB_TX1-: track 0.00 -> 19.8 mm, vias 0 -> 2
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Other:
- outline, holes or cut-outs redrawn
- board text added: "<- This GND is cooked"
- board text added: "Btw fix this curve"
