File: PiBoard.kicad_pcb (KiCad board)
At the start: 4 copper layers, 72.3 x 97.1 mm, 128 parts, among them IC1 TCAN337DCNR, IC2 TPS2557QDRBTQ1, IC3 LM74502HDDFR, IC4 AP64501QSP-13, IC5 TPS2557QDRBTQ1, IC8 TPS2557QDRBTQ1, J1 CarLVPowerConnector, J11 RTC Battery Port, J14 4x nano-fit, J2 Display Breakout, J3 2222, J5 USB_C_Receptacle_USB2.0_16P, J6 CarCANConnector, J7 HDMI_A_1.4, J8 CarCANConnector, J9 USB_A, Q2 NVMFWS1D7N04XMT1G, Q3 NVMFWS1D7N04XMT1G, SW1 SW_Push, SW2 SW_Push, U1 TPD1E05U06DYA, U13 CDSOT23-T24CAN, U14 MCP2515-E/STVAO, U2 TPD1E05U06DYA, U4 TPD1E05U06DYA, Y4 8 MHz

Commit message: frink4
Routing:
- net +5V: track 25.4 -> 22.3 mm, vias 2 -> 0
- net /CM5 GPIO/FAN_PWM: track 56.9 -> 56.7 mm, vias 4 -> 5
Changed lines of the file:
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@@
 		(net 1)
 	)
-	(via
-		(at 114.55 101.8)
-		(size 0.6)
-		(drill 0.3)
-		(layers "F.Cu" "B.Cu")
-		(free yes)
-		(net 1)
-	)
-	(via
-		(at 114.9 98.85)
-		(size 0.6)
-		(drill 0.3)
-		(layers "F.Cu" "B.Cu")
-		(free yes)
-		(net 1)
-	)
-	(segment
-		(start 114.9 98.85)
-		(end 114.9 101.45)
-		(width 0.5)
-		(layer "B.Cu")
-		(net 1)
-	)
-	(segment
-		(start 114.9 101.45)
-		(end 114.55 101.8)
-		(width 0.5)
-		(layer "B.Cu")
-		(net 1)
-	)
 	(segment
 		(start 132.65 96.9325)
@@
 	)
 	(segment
-		(start 113.65 95.45)
-		(end 111.8625 93.6625)
+		(start 111.8375 94.4)
+		(end 111.1 93.6625)
 		(width 0.2)
 		(layer "F.Cu")
@@
 	)
 	(segment
-		(start 113.65 96.75)
-		(end 113.65 95.45)
+		(start 112.185 94.4)
+		(end 111.8375 94.4)
 		(width 0.2)
 		(layer "F.Cu")
@@
 	)
 	(segment
-		(start 111.8625 93.6625)
-		(end 111.1 93.6625)
-		(width 0.2)
-		(layer "F.Cu")
-		(net 101)
-	)
-	(segment
 		(start 113.55 96.85)
 		(end 112.025 96.85)
@@
 	)
 	(via
+		(at 112.185 94.4)
+		(size 0.6)
+		(drill 0.3)
+		(layers "F.Cu" "B.Cu")
+		(net 101)
+	)
+	(via
 		(at 80.240325 114.898544)
 		(size 0.6)
@@
 	)
 	(segment
+		(start 112.185 94.4)
+		(end 113.65 95.865)
+		(width 0.2)
+		(layer "In2.Cu")
+		(net 101)
+	)
+	(segment
 		(start 110.7985 98.2765)
 		(end 95.351 113.724)
@@
 		(layer "In2.Cu")
 		(net 101)
+	)
+	(segment
+		(start 113.65 95.865)
+		(end 113.65 96.75)
+		(width 0.2)
+		(layer "In2.Cu")
+		(net 101)

Commit message: lak
Parts:
- removed C2: 100n, Capacitor_SMD:C_0603_1608Metric_Pad1.08x0.95mm_HandSolder
- removed D22: FAULT, LED_SMD:LED_0603_1608Metric_Pad1.05x0.95mm_HandSolder
- removed FB1: FerriteBead, Inductor_SMD:L_1206_3216Metric
- removed IC2: TPS2557QDRBTQ1, Controls_Pi:SON65P300X300X100-9N-D
- removed R100: 10k, Resistor_SMD:R_0603_1608Metric_Pad0.98x0.95mm_HandSolder
- removed R23: 1.5k, Resistor_SMD:R_0603_1608Metric_Pad0.98x0.95mm_HandSolder
- removed R5: 180k, Resistor_SMD:R_0603_1608Metric_Pad0.98x0.95mm_HandSolder
- removed U4: TPD1E05U06DYA, Diode_SMD:D_SOD-523
- moved C1 5.04 mm to (122.7, 97.5), turned to 180 degrees
- moved D3 4.27 mm to (122.7, 95.8)
- moved R3 4.27 mm to (125.2, 96.7)
- moved D8 3.52 mm to (124.7, 100.9)
- moved C3 1.70 mm to (109.5, 87.6)
- moved R13 1.70 mm to (107.1, 88.5)
- moved R14 1.70 mm to (107.1, 86.9)
- moved J5 0.57 mm to (129.0, 100.2)
- moved R16 0.57 mm to (132.6, 101.9)
- moved R18 0.57 mm to (132.6, 98.4)
Connections:
- C1 pad 1: +5V -> Net-(C1-Pad1)
- C18 pad 2: /Power Distribution/RPP_EN -> /Power Distribution/LV+
- C19 pad 1: /Power Distribution/RPP_EN -> /Power Distribution/LV+
- IC3 pad 1: /Power Distribution/RPP_EN -> /Power Distribution/LV+
- IC3 pad 5: /Power Distribution/RPP_EN -> /Power Distribution/LV+
- IC3 pad 8: +24V -> Net-(IC3-SRC)
- J5 pad A4: Net-(U4-I/O) -> Net-(C1-Pad1)
- J5 pad A9: Net-(U4-I/O) -> Net-(C1-Pad1)
- J5 pad B4: Net-(U4-I/O) -> Net-(C1-Pad1)
- J5 pad B9: Net-(U4-I/O) -> Net-(C1-Pad1)
- Q2 pad 1: Net-(Q2-Pad1) -> Net-(IC3-SRC)
- Q2 pad 2: Net-(Q2-Pad1) -> Net-(IC3-SRC)
- Q2 pad 3: Net-(Q2-Pad1) -> Net-(IC3-SRC)
- Q3 pad 1: Net-(Q2-Pad1) -> Net-(IC3-SRC)
- Q3 pad 2: Net-(Q2-Pad1) -> Net-(IC3-SRC)
- Q3 pad 3: Net-(Q2-Pad1) -> Net-(IC3-SRC)
- R3 pad 1: /High Speed/USB-C/VBUS_DBG -> Net-(C1-Pad1)
Routing:
- net /CM5 GPIO/GLOBAL_EN: track 154.5 -> 82.4 mm, vias 6 -> 3
- net Net-(C1-Pad1): track 0.00 -> 14.7 mm, vias 0 -> 2
- net /Power Distribution/LV+: track 0.00 -> 12.8 mm, vias 0 -> 2
- net GND: track 204.1 -> 193.5 mm, vias 167 -> 164
- net /Power Distribution/RPP_EN: track 9.83 -> 0.00 mm
- net Net-(IC2-ILIM): track 7.83 -> 0.00 mm, vias 2 -> 0
- net Net-(U4-I/O): track 4.88 -> 0.00 mm, vias 2 -> 0
- net /High Speed/USB_DBG_D-: track 35.3 -> 31.9 mm, vias 2 -> 0
- net +24V: track 3.33 -> 0.00 mm, vias 2 -> 0
- net /High Speed/USB_DBG_D+: track 35.6 -> 32.5 mm
- net Net-(IC3-SRC): track 0.00 -> 2.89 mm, vias 0 -> 2
- net /High Speed/USB-C/VBUS_DBG: track 2.18 -> 0.00 mm
- net Net-(IC3-OV): track 6.44 -> 4.51 mm
- net Net-(D22-K): track 1.83 -> 0.00 mm
- net Net-(D22-A): track 1.62 -> 0.00 mm
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- added copper zone on F.Cu, net Net-(IC3-SRC)
- removed copper zone on F.Cu, net /High Speed/USB-C/VBUS_DBG
- removed copper zone on F.Cu, net Net-(Q2-Pad1)
- removed copper zone on F.Cu, net Net-(U4-I/O)

Commit message: chang
Parts:
- added D20: VSSAF522-M3/H, UTSVT_Passives:MMDL101T1G, F.Cu at (117.0, 97.0)
- added R5: 1000, Resistor_SMD:R_0603_1608Metric_Pad0.98x0.95mm_HandSolder, F.Cu at (116.2, 90.7)
- H1, H2, H3, H4: footprint MountingHole:MountingHole_3mm -> MountingHole:MountingHole_3.2mm_M3
- U14: value MCP2515-E/STVAO -> MCP2515T-E/ST
- moved C24 8.80 mm to (124.3, 82.7)
- moved TP5 3.96 mm to (115.4, 73.2)
- moved C25 3.52 mm to (114.7, 82.6)
- moved C37 2.59 mm to (124.3, 93.1), turned to 0 degrees
- moved C36 1.39 mm to (116.3, 89.1)
- moved R34 1.39 mm to (116.3, 87.6)
- moved Y4 1.00 mm to (119.5, 81.7)
- moved U14 1.00 mm to (121.5, 88.3)
- moved H3 0.15 mm to (66.8, 154.3)
- moved H4 0.15 mm to (121.1, 154.3)
Connections:
- C36 pad 1: +3.3V -> Net-(C36-Pad1)
- R34 pad 2: +3.3V -> Net-(C36-Pad1)
Routing:
- net Net-(C36-Pad1): track 0.00 -> 3.75 mm
- net Net-(U14-OSC1): track 8.55 -> 7.13 mm
- net Net-(U14-OSC2): track 8.45 -> 7.14 mm
- net /CM5 GPIO/CAN_SPI_MISO: track 118.2 -> 119.5 mm
- net /CM5 GPIO/CAN_INTR: track 74.0 -> 75.1 mm
- net /CM5 GPIO/CAN_SPI_CS: track 78.1 -> 79.1 mm
- net /CM5 GPIO/CAN_SPI_MOSI: track 133.9 -> 135.0 mm
- net +3.3V: track 221.4 -> 222.4 mm
- net GND: track 193.5 -> 194.5 mm, vias 164 -> 167
- net /CM5 GPIO/CAN_SPI_CLK: track 114.0 -> 114.7 mm
Other:
- board text added: "Need to fix impedence matching"

Commit message: imp
Routing:
- net /High Speed/USB_HUB_RX1+: track 16.3 -> 15.6 mm
- net /High Speed/USB_HUB_RX1-: track 16.3 -> 15.6 mm
- net /High Speed/HDMI0_HOTPLUG: track 30.2 -> 29.7 mm
Other:
- board text added: "Impedence is ok? HDMI: 0.15w, 0.126sp USB: 0.17w, 0.1sp"
- board text removed: "Need to fix impedence matching"

Commit message: fjfdsfdslk
Parts:
- moved D19 0.35 mm to (114.7, 112.3)
Routing:
- net GND: track 194.5 -> 197.1 mm, vias 167 -> 205
- net /High Speed/USB_HUB_D+: track 17.1 -> 18.2 mm
- net Net-(J9-DRAIN): track 25.7 -> 24.5 mm

Commit message: P/Ns
Parts:
- C18: value 1u -> 1uF
- C19: value 220n -> 220nF
- C27: value 10u -> 10uF
- C3: value 0.1u -> 100n
- C56: value 10n -> 10nF
- C59: value 2.7n -> 2.7nF
- C60: value 33p -> 33pF
- C61, C8, C9: value 22u -> 22uF
- L2: value 4.7 u -> 4.7uH
- R1, R15, R2, R20, R25, R33, R42: value 700 -> 100
- R21, R22, R3, R45, R8: value 1.5k -> 200
- R44: value 10k -> 1.5k; footprint Resistor_SMD:R_0603_1608Metric_Pad0.98x0.95mm_HandSolder -> Resistor_SMD:R_0805_2012Metric_Pad1.20x1.40mm_HandSolder
- R5: value 1000 -> 1k
- moved R44 0.18 mm to (94.4, 88.3)
