File: CM5_GPIO.kicad_sch (KiCad schematic)
At the start: 28 parts, among them J11 RTC Battery Port, J12 RTC Battery Conn, J14 4x nano-fit, J3 2222, SW1 SW_Push, SW2 SW_Push

Commit message: rrrrrrrr
Parts:
- added TP5: TestPoint, TestPoint:TestPoint_Pad_2.0x2.0mm, symbol Connector:TestPoint
Connections:
- net +3.3V: now also TP5.1
Changed lines of the file:
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@@
 	)
 	(symbol
+		(lib_id "Connector:TestPoint")
+		(at 21.59 120.65 180)
+		(unit 1)
+		(exclude_from_sim no)
+		(in_bom yes)
+		(on_board yes)
+		(dnp no)
+		(property "Reference" "TP5"
+			(at 18.923 123.0122 90)
+			(effects
+				(font
+					(size 1.27 1.27)
+				)
+				(justify left)
+			)
+		)
+		(property "Value" "TestPoint"
+			(at 24.003 117.9322 90)
+			(effects
+				(font
+					(size 1.27 1.27)
+				)
+				(justify left)
+			)
+		)
+		(property "Footprint" "TestPoint:TestPoint_Pad_2.0x2.0mm"
+			(at 16.51 120.65 0)
+			(effects
+				(font
+					(size 1.27 1.27)
+				)
+				(hide yes)
+			)
+		)
+		(property "Datasheet" "~"
+			(at 16.51 120.65 0)
+			(effects
+				(font
+					(size 1.27 1.27)
+				)
+				(hide yes)
+			)
+		)
+		(property "Description" "test point"
+			(at 21.59 120.65 0)
+			(effects
+				(font
+					(size 1.27 1.27)
+				)
+				(hide yes)
+			)
+		)
+		(pin "1"
+		)
+		(instances
+			(project "PiBoard"
+				(path "/e4d65698-b8ec-4bf6-9f2b-a5010377155a/353ee88d-a044-4c9d-80a8-948975426026"
+					(reference "TP5")
+					(unit 1)
+				)
+			)
+		)
+	)
+	(symbol
 		(lib_id "power:GND")
 		(at 241.3 72.39 0)
@@
 			)
 		)
-		(property "Datasheet" ""
+		(property "Datasheet" "https://storage.raspberrypi.com/product-information/hawl3l9kl3xwo8tj8e2msztrus1n?response-content-disposition=inline%3B%20filename%3D%22RP-008180-DS-cm5-datasheet.pdf%22%3B%20filename%2A%3DUTF-8%27%27RP-008180-DS-cm5-datasheet.pdf&response-content-type=application%2Fpdf&X-Amz-Algorithm=AWS4-HMAC-SHA256&X-Amz-Credential=product-information%2F20251004%2Feu-west-1%2Fs3%2Faws4_request&X-Amz-Date=20251004T180850Z&X-Amz-Expires=172800&X-Amz-SignedHeaders=host&X-Amz-Signature=be9dd03b4fc44e5a401ffdce01adaaf5f36a0d9794c56bc665f3d3971a12888a"
 			(at 219.71 116.84 0)
 			(effects
@@
 		)
 		(instances
-			(project ""
+			(project "PiBoard"
 				(path "/e4d65698-b8ec-4bf6-9f2b-a5010377155a/353ee88d-a044-4c9d-80a8-948975426026"
 					(reference "#PWR07")
@@
 		)
 		(instances
-			(project ""
+			(project "PiBoard"
 				(path "/e4d65698-b8ec-4bf6-9f2b-a5010377155a/353ee88d-a044-4c9d-80a8-948975426026"
 					(reference "#PWR05")
@@
 					(unit 1)
 				)
+			)
+		)
+	)
+	(symbol
+		(lib_id "power:+3.3V")
+		(at 21.59 120.65 0)
+		(unit 1)
+		(exclude_from_sim no)
+		(in_bom yes)
+		(on_board yes)
+		(dnp no)
+		(fields_autoplaced yes)
+		(property "Reference" "#PWR0115"
+			(at 21.59 124.46 0)
+			(effects
+				(font
+					(size 1.27 1.27)
+				)
+				(hide yes)
+			)
+		)
+		(property "Value" "+3.3V"
+			(at 21.59 115.57 0)
+			(effects
+				(font
+					(size 1.27 1.27)
+				)
+			)
+		)
+		(property "Footprint" ""
+			(at 21.59 120.65 0)
+			(effects
+				(font
+					(size 1.27 1.27)
+				)
+				(hide yes)
+			)
+		)
+		(property "Datasheet" ""
+			(at 21.59 120.65 0)
+			(effects
+				(font
+					(size 1.27 1.27)
+				)
+				(hide yes)
+			)
+		)
+		(property "Description" "Power symbol creates a global label with name \"+3.3V\""
+			(at 21.59 120.65 0)
+			(effects
+				(font
+					(size 1.27 1.27)
+				)
+				(hide yes)
+			)
+		)
+		(pin "1"
+		)
+		(instances
+			(project "PiBoard"
+				(path "/e4d65698-b8ec-4bf6-9f2b-a5010377155a/353ee88d-a044-4c9d-80a8-948975426026"
+					(reference "#PWR0115")
+					(unit 1)
+				)

Commit message: I hate my life
Parts:
- added R27: 10K, Resistor_SMD:R_0603_1608Metric_Pad0.98x0.95mm_HandSolder, symbol Device:R
- C22, C23: footprint Capacitor_SMD:C_0603_1608Metric -> Capacitor_SMD:C_0603_1608Metric_Pad1.08x0.95mm_HandSolder
- D1, D13, D14, D16, D2, D5: footprint LED_SMD:LED_0603_1608Metric -> LED_SMD:LED_0603_1608Metric_Pad1.05x0.95mm_HandSolder
- R1, R42: value 1k -> 700; footprint Resistor_SMD:R_0603_1608Metric -> Resistor_SMD:R_0603_1608Metric_Pad0.98x0.95mm_HandSolder
- R15, R17, R19, R20, R25, R33: footprint Resistor_SMD:R_0603_1608Metric -> Resistor_SMD:R_0603_1608Metric_Pad0.98x0.95mm_HandSolder
- R4: value 10K 1% -> 10K; footprint Resistor_SMD:R_0603_1608Metric -> Resistor_SMD:R_0603_1608Metric_Pad0.98x0.95mm_HandSolder
Connections:
- net +3.3V: now also R27.2
- net FAN_TACHO: now also R27.1
Other:
- note added: "*Prob will not have to be placed"
- note added: "CM5IO: Pullup added for Fans that don't have a strong internal pullup"
- note removed: "R2 : Pullup added for Fans that don't have a strong internal pullup"
- moved on the sheet: J14, R4

Commit message: rrr
Other:
- note added: "Jus for looks man"
Changed lines of the file:
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@@
+		)
+	)
+	(text "Jus for looks man"
+		(exclude_from_sim no)
+		(at 247.142 157.226 0)
+		(effects
+			(font
+				(size 1.27 1.27)
+			)
 		)
 	)

Commit message: frank
Connections:
- net +24V: no longer J14.1 (Pin_1)
- net +5V: now also J14.1 (Pin_1)
Changed lines of the file:
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@@
 			)
 		)
-		(property "Value" "+24V"
+		(property "Value" "+5V"
 			(at 261.112 100.584 0)
 			(effects

Commit message: Copy of I hate my life pt2.5 final final (3)
Connections:
- net GPIO13: now also R33.2; no longer R20.2
- net GPIO19: now also R20.2; no longer R15.2
- net GPIO26: now also R15.2; no longer R33.2
Changed lines of the file:
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@@
 		)
 	)
-	(label "GPIO13"
+	(label "GPIO19"
 		(at 175.26 44.45 180)
 		(effects
@@
 		)
 	)
+	(label "GPIO13"
+		(at 200.66 44.45 180)
+		(effects
+			(font
+				(size 1.27 1.27)
+			)
+			(justify right bottom)
+		)
+	)
 	(label "GPIO26"
 		(at 30.48 62.23 0)
@@
 	)
 	(label "GPIO26"
-		(at 200.66 44.45 180)
+		(at 187.96 44.45 180)
 		(effects
 			(font
@@
 		)
 	)
-	(label "GPIO19"
-		(at 187.96 44.45 180)
-		(effects
-			(font
-				(size 1.27 1.27)
-			)
-			(justify right bottom)
-		)
-	)

Commit message: my life could not be worse right now
Other:
- note added: "Pull low"
Changed lines of the file:
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@@
 		)
 	)
+	(text "Pull low"
+		(exclude_from_sim no)
+		(at 156.718 100.33 0)
+		(effects
+			(font
+				(size 1.27 1.27)
+			)
+		)
+	)
 	(text "RTC BATT"
 		(exclude_from_sim no)
@@
 			)
 		)
-		(property "Datasheet" "https://storage.raspberrypi.com/product-information/hawl3l9kl3xwo8tj8e2msztrus1n?response-content-disposition=inline%3B%20filename%3D%22RP-008180-DS-cm5-datasheet.pdf%22%3B%20filename%2A%3DUTF-8%27%27RP-008180-DS-cm5-datasheet.pdf&response-content-type=application%2Fpdf&X-Amz-Algorithm=AWS4-HMAC-SHA256&X-Amz-Credential=product-information%2F20251004%2Feu-west-1%2Fs3%2Faws4_request&X-Amz-Date=20251004T180850Z&X-Amz-Expires=172800&X-Amz-SignedHeaders=host&X-Amz-Signature=be9dd03b4fc44e5a401ffdce01adaaf5f36a0d9794c56bc665f3d3971a12888a"
+		(property "Datasheet" "https://pip-assets.raspberrypi.com/categories/944-raspberry-pi-compute-module-5/documents/RP-008180-DS-6-cm5-datasheet.pdf?disposition=inline"
 			(at 219.71 116.84 0)
 			(effects

Commit message: frink
Parts:
- R17, R19: value 10k -> 1k
Changed lines of the file:
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@@
 			)
 		)
-		(property "Value" "10k"
-			(at 156.972 111.76 90)
+		(property "Value" "1k"
+			(at 156.21 111.76 90)
 			(effects
 				(font
@@
 			)
 		)
-		(property "Value" "10k"
-			(at 156.972 71.12 90)
+		(property "Value" "1k"
+			(at 156.21 71.12 90)
 			(effects
 				(font

Commit message: chang
Parts:
- added D20: VSSAF522-M3/H, UTSVT_Passives:MMDL101T1G, symbol Diode:C3D25170H
Connections:
- net +5V: now also D20.1 (K)
- net GND: now also D20.2 (A)
Changed lines of the file:
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@@
 	(text "FAN connector\n"
 		(exclude_from_sim no)
-		(at 256.54 120.904 0)
+		(at 259.588 99.314 0)
 		(effects
 			(font
@@
 	)
 	(junction
+		(at 257.81 100.33)
+		(diameter 0)
+		(color 0 0 0 0)
+	)
+	(junction
 		(at 180.34 25.4)
 		(diameter 0)
@@
 	)
 	(junction
+		(at 257.81 115.57)
+		(diameter 0)
+		(color 0 0 0 0)
+	)
+	(junction
 		(at 43.18 72.39)
 		(diameter 0)
@@
 	(wire
 		(pts
+			(xy 267.97 100.33) (xy 257.81 100.33)
+		)
+		(stroke
+			(width 0)
+			(type default)
+		)
+	)
+	(wire
+		(pts
 			(xy 224.79 111.76) (xy 238.76 111.76)
 		)
@@
 	(wire
 		(pts
+			(xy 257.81 115.57) (xy 267.97 115.57)
+		)
+		(stroke
+			(width 0)
+			(type default)
+		)
+	)
+	(wire
+		(pts
 			(xy 119.38 148.59) (xy 105.41 148.59)
 		)
@@
 	(wire
 		(pts
-			(xy 257.81 104.14) (xy 257.81 102.87)
+			(xy 257.81 100.33) (xy 257.81 104.14)
 		)
 		(stroke
@@
 	(wire
 		(pts
+			(xy 257.81 97.79) (xy 257.81 100.33)
+		)
+		(stroke
+			(width 0)
+			(type default)
+		)
+	)
+	(wire
+		(pts
 			(xy 106.68 41.91) (xy 106.68 49.53)
 		)
@@
 	(wire
 		(pts
+			(xy 267.97 104.14) (xy 267.97 100.33)
+		)
+		(stroke
+			(width 0)
+			(type default)
+		)
+	)
+	(wire
+		(pts
 			(xy 255.27 48.26) (xy 266.7 48.26)
 		)
@@
 	(wire
 		(pts
+			(xy 267.97 115.57) (xy 267.97 111.76)
+		)
+		(stroke
+			(width 0)
+			(type default)
+		)
+	)
+	(wire
+		(pts
 			(xy 43.18 97.79) (xy 44.45 97.79)
 		)
@@
 	(wire
 		(pts
-			(xy 257.81 109.22) (xy 257.81 113.03)
+			(xy 257.81 109.22) (xy 257.81 115.57)
 		)
 		(stroke
@@
 	(wire
 		(pts
+			(xy 257.81 115.57) (xy 257.81 118.11)
+		)
+		(stroke
+			(width 0)
+			(type default)
+		)
+	)
+	(wire
+		(pts
 			(xy 43.18 115.57) (xy 43.18 125.73)
 		)
@@
 	(symbol
 		(lib_id "power:GND")
-		(at 257.81 113.03 0)
+		(at 257.81 118.11 0)
 		(unit 1)
 		(exclude_from_sim no)
@@
 		(dnp no)
 		(property "Reference" "#PWR037"
-			(at 257.81 119.38 0)
+			(at 257.81 124.46 0)
 			(effects
 				(font
@@
 		)
 		(property "Value" "GND"
-			(at 257.937 117.4242 0)
+			(at 257.937 122.5042 0)
 			(effects
 				(font
@@
 		)
 		(property "Footprint" ""
-			(at 257.81 113.03 0)
+			(at 257.81 118.11 0)
 			(effects
 				(font
@@
 		)
 		(property "Datasheet" ""
-			(at 257.81 113.03 0)
+			(at 257.81 118.11 0)
 			(effects
 				(font
@@
 		)
 		(property "Description" "Power symbol creates a global label with name \"GND\" , ground"
-			(at 257.81 113.03 0)
+			(at 257.81 118.11 0)
 			(effects
 				(font
@@
 		(dnp no)
 		(property "Reference" "J14"
-			(at 262.255 114.935 0)
+			(at 262.382 101.854 0)
 			(effects
 				(font
@@
 				)
 				(justify left)
+				(hide yes)
 			)
 		)
@@
 	(symbol
 		(lib_id "power:+12V")
-		(at 257.81 102.87 0)
+		(at 257.81 97.79 0)
 		(unit 1)
 		(exclude_from_sim no)
@@
 		(dnp no)
 		(property "Reference" "#PWR039"
-			(at 257.81 106.68 0)
+			(at 257.81 101.6 0)
 			(effects
 				(font
@@
 		)
 		(property "Value" "+5V"
-			(at 261.112 100.584 0)
+			(at 261.112 95.504 0)
 			(effects
 				(font
@@
 		)
 		(property "Footprint" ""
-			(at 257.81 102.87 0)
+			(at 257.81 97.79 0)
 			(effects
 				(font
@@
 		)
 		(property "Datasheet" ""
-			(at 257.81 102.87 0)
+			(at 257.81 97.79 0)
 			(effects
 				(font
@@
 		)
 		(property "Description" "Power symbol creates a global label with name \"+12V\""
-			(at 257.81 102.87 0)
+			(at 257.81 97.79 0)
 			(effects
 				(font
@@
 					(unit 1)
 				)
+			)
+		)
+	)
+	(symbol
+		(lib_id "Diode:C3D25170H")
+		(at 267.97 107.95 270)
+		(unit 1)
+		(exclude_from_sim no)
+		(in_bom yes)
+		(on_board yes)
+		(dnp no)
+		(property "Reference" "D20"
+			(at 270.256 105.41 90)
+			(effects
+				(font
+					(size 1.27 1.27)
+				)
+				(justify left)
+			)
+		)
+		(property "Value" "VSSAF522-M3/H"
+			(at 271.272 106.426 0)
+			(effects
+				(font
+					(size 1.27 1.27)
+				)
+				(justify left)
+			)
+		)
+		(property "Footprint" "UTSVT_Passives:MMDL101T1G"
+			(at 263.525 107.95 0)
+			(effects
+				(font
+					(size 1.27 1.27)
+				)
+				(hide yes)
+			)
+		)
+		(property "Datasheet" "https://www.mouser.com/ProductDetail/Vishay-General-Semiconductor/VSSAF522-M3-H?qs=UkDUCjYnTB00gpgD%2Fb%2Fw%252BA%3D%3D"
+			(at 267.97 107.95 0)
+			(effects
+				(font
+					(size 1.27 1.27)
+				)
+				(hide yes)
+			)
+		)
+		(property "Description" ""
+			(at 267.97 107.95 0)
+			(effects
+				(font
+					(size 1.27 1.27)
+				)
+				(hide yes)
+			)
+		)
+		(property "Manufactuerer" "Vishay General Semiconductor "
+			(at 267.97 107.95 90)
+			(effects
+				(font
+					(size 1.27 1.27)
+				)
+				(hide yes)
+			)
+		)
+		(property "P/N" "VSSAF522-M3/H"
+			(at 267.97 107.95 90)
+			(effects
+				(font
+					(size 1.27 1.27)
+				)
+				(hide yes)
+			)
+		)
+		(pin "1"
+		)
+		(pin "2"
+		)
+		(instances
+			(project "PiBoard"
+				(path "/e4d65698-b8ec-4bf6-9f2b-a5010377155a/353ee88d-a044-4c9d-80a8-948975426026"
+					(reference "D20")
+					(unit 1)
+				)
