File: CM5_GPIO.kicad_sch (KiCad schematic)
At the start: 31 parts, among them J11 RTC Battery Port, J12 RTC Battery Conn, J14 4x nano-fit, J3 2222, SW1 SW_Push, SW2 SW_Push

Commit message: P/Ns
Parts:
- C22, C23: P/N C0805C104M5RACTU -> MLASH168SB7104KTNA01
- D1, D13, D16, D5: P/N APTD2012LCGCK -> 150060VS55040
- D14: P/N APTD2012LCGCK -> LS Q976.01-N1Q2-1
- D2: P/N APTD2012LSURCK -> 150060VS55040
- J14: value 4x nano-fit -> Fan Header; P/N (none) -> SHBM04B-SRSS-TB
- J3: value 2222 -> RPI Pin-Header
- Module2: P/N (none) -> 10164227-1001A1RLF
- R1, R15, R20, R33, R42: value 700 -> 100; P/N CRCW08051K00FKEAC -> CRCW0603100RFKEA
- R17, R19: P/N CRCW08051K00FKEAC -> CRCW06031K00FKEI
- R25: value 700 -> 100; P/N ERJ-P06F7150V -> CRCW0603100RFKEA
- R27, R4: value 10K -> 10k; P/N (none) -> CRCW060310K0FKEI
Other:
- note added: "fwd cur: ~13ma fwd volt: ~2V R: ~100"
- note removed: "fwd cur: ~2ma fwd volt: ~2V R: ~650-700"

Commit message: silkscreen n shit
Parts:
- removed S1, S2: DPDT Switch, Controls_Pi:CLSB22B12T, symbol CL-SB-22B-12T:CL-SB-22B-12T
- added JP2, JP3, JP4, JP5: Jumper_2_Open, Connector_PinHeader_2.54mm:PinHeader_1x02_P2.54mm_Vertical, symbol Jumper:Jumper_2_Open
Connections:
- net BT_Disable: now also JP3.2 (B)
- net EEPROM_nWP: now also JP5.2 (B)
- net GND: now also JP2.1 (A), JP3.1 (A), JP4.1 (A), JP5.1 (A)
- net WiFi_Disable: now also JP2.2 (B)
- net nRPIBOOT: now also JP4.2 (B)
- no-connect marks 31 -> 27
Other:
- note removed: "Double check this for sanity"
- note removed: "Ready EMMC for flash"
- note removed: "Wireless EN"

Commit message: jlc shit
Parts:
- BT2, J11, J12, J14, J3, JP2, JP3, JP4, JP5, SW1, SW2, TP4, TP5: JLC (none) -> N/A
- C22, C23: JLC (none) -> C14663
- D1, D13, D16, D2, D5: JLC (none) -> C2289
- D14: JLC (none) -> C2286
- D20: JLC (none) -> C20039242
- Module2: JLC (none) -> C6782225
- R1, R15, R20, R25, R33, R42: JLC (none) -> C22775
- R17, R19: JLC (none) -> C21190
- R27, R4: JLC (none) -> C25804

Commit message: poop
Parts:
- removed TP4: TestPoint, TestPoint:TestPoint_Pad_2.0x2.0mm, symbol Connector:TestPoint
- D20: value VSSAF522-M3/H -> SMF5.0A; footprint UTSVT_Passives:MMDL101T1G -> Diode_SMD:D_SOD-123; JLC C20039242 -> C193402; Manufactuerer Vishay General Semiconductor -> (none); P/N VSSAF522-M3/H -> SMF5.0A
- R4: now not fitted
- SW1, SW2: footprint Button_Switch_SMD:SW_SPST_B3SL-1002P -> CM5IO:TL3365AF180QG; JLC N/A -> C2886926; P/N 653-B3SL-1002P -> TL3365AF180QG
Other:
- note added: "Change button P/N to PSOM"
- note added: "Fix"
Changed lines of the file:
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@@
 		)
 	)
+	(text "Change button P/N\nto PSOM"
+		(exclude_from_sim no)
+		(at 194.056 79.502 0)
+		(effects
+			(font
+				(size 3 3)
+				(thickness 0.254)
+				(bold yes)
+			)
+		)
+	)
 	(text "Global En"
 		(exclude_from_sim no)
@@
 		)
 	)
+	(text "Fix"
+		(exclude_from_sim no)
+		(at 278.638 109.22 0)
+		(effects
+			(font
+				(size 3 3)
+				(thickness 0.6)
+				(bold yes)
+			)
+		)
+	)
 	(text "For USB\nPD"
 		(exclude_from_sim no)
@@
 			)
 		)
-		(property "Footprint" "Button_Switch_SMD:SW_SPST_B3SL-1002P"
+		(property "Footprint" "CM5IO:TL3365AF180QG"
 			(at 146.05 68.58 0)
 			(effects
@@
 			)
 		)
-		(property "P/N" "653-B3SL-1002P"
+		(property "P/N" "TL3365AF180QG"
 			(at 146.05 73.66 0)
 			(effects
@@
 			)
 		)
-		(property "JLC" "N/A"
+		(property "JLC" "C2886926"
 			(at 146.05 73.66 0)
 			(effects
@@
 			)
 		)
-		(property "Footprint" "Button_Switch_SMD:SW_SPST_B3SL-1002P"
+		(property "Footprint" "CM5IO:TL3365AF180QG"
 			(at 146.05 109.22 0)
 			(effects
@@
 			)
 		)
-		(property "P/N" "653-B3SL-1002P"
+		(property "P/N" "TL3365AF180QG"
 			(at 146.05 114.3 0)
 			(effects
@@
 			)
 		)
-		(property "JLC" "N/A"
+		(property "JLC" "C2886926"
 			(at 146.05 114.3 0)
 			(effects
@@
 		(in_bom yes)
 		(on_board yes)
-		(dnp no)
+		(dnp yes)
 		(property "Reference" "R4"
 			(at 252.222 101.4984 0)
@@
 	)
 	(symbol
-		(lib_id "power:+3.3V")
-		(at 26.67 163.83 0)
-		(unit 1)
-		(exclude_from_sim no)
-		(in_bom yes)
-		(on_board yes)
-		(dnp no)
-		(property "Reference" "#PWR018"
-			(at 26.67 167.64 0)
-			(effects
-				(font
-					(size 1.27 1.27)
-				)
-				(hide yes)
-			)
-		)
-		(property "Value" "+1.8V"
-			(at 26.416 160.02 0)
-			(effects
-				(font
-					(size 1.27 1.27)
-				)
-			)
-		)
-		(property "Footprint" ""
-			(at 26.67 163.83 0)
-			(effects
-				(font
-					(size 1.27 1.27)
-				)
-				(hide yes)
-			)
-		)
-		(property "Datasheet" ""
-			(at 26.67 163.83 0)
-			(effects
-				(font
-					(size 1.27 1.27)
-				)
-				(hide yes)
-			)
-		)
-		(property "Description" "Power symbol creates a global label with name \"+3.3V\""
-			(at 26.67 163.83 0)
-			(effects
-				(font
-					(size 1.27 1.27)
-				)
-				(hide yes)
-			)
-		)
-		(pin "1"
-		)
-		(instances
-			(project "PiBoard"
-				(path "/e4d65698-b8ec-4bf6-9f2b-a5010377155a/353ee88d-a044-4c9d-80a8-948975426026"
-					(reference "#PWR018")
-					(unit 1)
-				)
-			)
-		)
-	)
-	(symbol
 		(lib_id "Device:R")
 		(at 238.76 106.68 180)
@@
 	)
 	(symbol
-		(lib_id "Connector:TestPoint")
-		(at 26.67 163.83 180)
-		(unit 1)
-		(exclude_from_sim no)
-		(in_bom yes)
-		(on_board yes)
-		(dnp no)
-		(property "Reference" "TP4"
-			(at 24.003 166.1922 90)
-			(effects
-				(font
-					(size 1.27 1.27)
-				)
-				(justify left)
-			)
-		)
-		(property "Value" "TestPoint"
-			(at 29.083 161.1122 90)
-			(effects
-				(font
-					(size 1.27 1.27)
-				)
-				(justify left)
-			)
-		)
-		(property "Footprint" "TestPoint:TestPoint_Pad_2.0x2.0mm"
-			(at 21.59 163.83 0)
-			(effects
-				(font
-					(size 1.27 1.27)
-				)
-				(hide yes)
-			)
-		)
-		(property "Datasheet" "~"
-			(at 21.59 163.83 0)
-			(effects
-				(font
-					(size 1.27 1.27)
-				)
-				(hide yes)
-			)
-		)
-		(property "Description" "test point"
-			(at 26.67 163.83 0)
-			(effects
-				(font
-					(size 1.27 1.27)
-				)
-				(hide yes)
-			)
-		)
-		(property "Data" ""
-			(at 26.67 163.83 90)
-			(effects
-				(font
-					(size 1.27 1.27)
-				)
-				(hide yes)
-			)
-		)
-		(property "JLC" "N/A"
-			(at 26.67 163.83 90)
-			(effects
-				(font
-					(size 1.27 1.27)
-				)
-				(hide yes)
-			)
-		)
-		(pin "1"
-		)
-		(instances
-			(project "PiBoard"
-				(path "/e4d65698-b8ec-4bf6-9f2b-a5010377155a/353ee88d-a044-4c9d-80a8-948975426026"
-					(reference "TP4")
-					(unit 1)
-				)
-			)
-		)
-	)
-	(symbol
 		(lib_id "Device:LED")
 		(at 140.97 30.48 90)
@@
 			)
 		)
-		(property "Value" "VSSAF522-M3/H"
+		(property "Value" "SMF5.0A"
 			(at 271.272 106.426 0)
 			(effects
@@
 			)
 		)
-		(property "Footprint" "UTSVT_Passives:MMDL101T1G"
+		(property "Footprint" "Diode_SMD:D_SOD-123"
 			(at 263.525 107.95 0)
 			(effects
@@
 			)
 		)
-		(property "Datasheet" "https://www.mouser.com/ProductDetail/Vishay-General-Semiconductor/VSSAF522-M3-H?qs=UkDUCjYnTB00gpgD%2Fb%2Fw%252BA%3D%3D"
+		(property "Datasheet" "https://www.littelfuse.com/assetdocs/tvs-diodes-smf-datasheet?assetguid=7eb8a5b6-bdd0-4561-8f19-0c3cc6f9b2af"
 			(at 267.97 107.95 0)
 			(effects
@@
 			)
 		)
-		(property "Manufactuerer" "Vishay General Semiconductor "
+		(property "Manufactuerer" ""
 			(at 267.97 107.95 90)
 			(effects
@@
 			)
 		)
-		(property "P/N" "VSSAF522-M3/H"
+		(property "P/N" "SMF5.0A"
 			(at 267.97 107.95 90)
 			(effects
@@
 			)
 		)
-		(property "JLC" "C20039242"
+		(property "JLC" "C193402"
 			(at 267.97 107.95 90)
 			(effects

Commit message: poop
Parts:
- removed D20: SMF5.0A, Diode_SMD:D_SOD-123, symbol Diode:C3D25170H
- added D6: PTVS6V0S1UR, Diode_SMD:D_SOD-123, symbol Diode:MBR0520
- added F3: RFuse, Fuse:Fuse_1206_3216Metric_Pad1.42x1.75mm_HandSolder, symbol Device:Fuse
Connections:
- net +5V: now also F3.2; no longer Module2.77 (+5v_(Input)), Module2.79 (+5v_(Input)), Module2.81 (+5v_(Input)), Module2.83 (+5v_(Input)), Module2.85 (+5v_(Input)), Module2.87 (+5v_(Input))
- net GND: now also D6.2 (A)
- new net CM5PWR: D6.1 (K), F3.1, Module2.77 (+5v_(Input)), Module2.79 (+5v_(Input)), Module2.81 (+5v_(Input)), Module2.83 (+5v_(Input)), Module2.85 (+5v_(Input)), Module2.87 (+5v_(Input))
Other:
- note added: "Because I am *retarded*"
- note removed: "Fix"

Commit message: poop
Other:
- note removed: "Change button P/N to PSOM"
Changed lines of the file:
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@@
-		)
-	)
-	(text "Change button P/N\nto PSOM"
-		(exclude_from_sim no)
-		(at 194.056 79.502 0)
-		(effects
-			(font
-				(size 3 3)
-				(thickness 0.254)
-				(bold yes)
-			)
 		)
 	)
