File: CM5_GPIO.kicad_sch (KiCad schematic)
At the start: 33 parts, among them J11 RTC Battery Port, J12 RTC Battery Conn, J14 Fan Header, J3 RPI Pin-Header, SW1 SW_Push, SW2 SW_Push

Commit message: Mika (#2)
* poop

* poop

* poop

* poop

* poop

* ideal diode circuit protection on usbc

* addressing mika's comments

* mika changes

* mika fixes

* mika changes

* poop

* mika changes

* poop

* poop

---------

Co-authored-by: Frank Li <fxl77@my.utexas.edu>
Parts:
- removed D20: VSSAF522-M3/H, UTSVT_Passives:MMDL101T1G, symbol Diode:C3D25170H
- removed TP4: TestPoint, TestPoint:TestPoint_Pad_2.0x2.0mm, symbol Connector:TestPoint
- added D6: PTVS6V0S1UR, Diode_SMD:D_SOD-123, symbol Diode:MBR0520
- added F3: RFuse, Fuse:Fuse_1206_3216Metric_Pad1.42x1.75mm_HandSolder, symbol Device:Fuse
- R4: now not fitted
- SW1, SW2: footprint Button_Switch_SMD:SW_SPST_B3SL-1002P -> CM5IO:TL3365AF180QG; JLC N/A -> C2886926; P/N 653-B3SL-1002P -> TL3365AF180QG
Connections:
- net +5V: now also F3.2; no longer Module2.77 (+5v_(Input)), Module2.79 (+5v_(Input)), Module2.81 (+5v_(Input)), Module2.83 (+5v_(Input)), Module2.85 (+5v_(Input)), Module2.87 (+5v_(Input))
- net GND: now also D6.2 (A)
- new net CM5PWR: D6.1 (K), F3.1, Module2.77 (+5v_(Input)), Module2.79 (+5v_(Input)), Module2.81 (+5v_(Input)), Module2.83 (+5v_(Input)), Module2.85 (+5v_(Input)), Module2.87 (+5v_(Input))
Other:
- note added: "Because I am *retarded*"
