File: PWR_Distribution.kicad_sch (KiCad schematic)
At the start: 33 parts, among them IC3 LM74502HDDFR, IC4 AP64501QSP-13, J1 CarLVPowerConnector, J2 Display Breakout, Q1 PSMN8R5-40MSDX

Commit message: rrrrrrrr
Parts:
- added F1: 1A, symbol Device:Fuse
- added TP1, TP2: TestPoint, TestPoint:TestPoint_Pad_2.0x2.0mm, symbol Connector:TestPoint
Connections:
- net +24V: now also F1.2, TP1.1; no longer J2.1 (+24V)
- net +5V: now also TP2.1
- new net: F1.1, J2.1 (+24V)
Other:
- note removed: "fuse here"
- moved on the sheet: TP3

Commit message: Schem done? [plz full review], redoing layout
Parts:
- F1: footprint (none) -> Fuse:Fuse_0805_2012Metric; P/N (none) -> MFU0805FF01000P500
Other:
- note added: "Display PWR"
- moved on the sheet: F1, J2
Changed lines of the file:
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@@
 		)
 	)
+	(rectangle
+		(start 193.04 44.45)
+		(end 240.03 85.09)
+		(stroke
+			(width 0)
+			(type default)
+		)
+		(fill
+			(type none)
+		)
+	)
 	(text "Est. max power draw (CM5) \n= 10W (pi) + 1.5W (HDMI) + 0.6W (CAN) \n= ~12.1W (rest of board draws negligible power)\n"
 		(exclude_from_sim no)
@@
 		)
 	)
+	(text "Display PWR"
+		(exclude_from_sim no)
+		(at 215.9 50.546 0)
+		(effects
+			(font
+				(size 2 2)
+				(thickness 0.25)
+			)
+		)
+	)
 	(text "Est. max power draw \n= 15W (pi) + 1.5W (HDMI) + 0.6W (CAN) \n= 21.6W (rest of board draws negligible power)\n"
 		(exclude_from_sim no)
@@
 	(text "Power"
 		(exclude_from_sim no)
-		(at 261.366 26.416 0)
+		(at 216.154 24.384 0)
 		(effects
 			(font
-				(size 2.54 2.54)
+				(size 3 3)
 				(thickness 0.508)
 				(bold yes)
@@
 	(wire
 		(pts
-			(xy 215.9 57.15) (xy 219.71 57.15)
+			(xy 215.9 67.31) (xy 219.71 67.31)
 		)
 		(stroke
@@
 	(wire
 		(pts
-			(xy 227.33 57.15) (xy 231.14 57.15)
+			(xy 227.33 67.31) (xy 231.14 67.31)
 		)
 		(stroke
@@
 	(hierarchical_label "+5V_PWR"
 		(shape input)
-		(at 219.71 26.67 270)
+		(at 181.61 135.89 270)
 		(effects
 			(font
@@
 	(hierarchical_label "+24V_PWR"
 		(shape output)
-		(at 212.09 26.67 270)
+		(at 173.99 135.89 270)
 		(effects
 			(font
@@
 	(symbol
 		(lib_id "power:+12V")
-		(at 212.09 26.67 0)
+		(at 173.99 135.89 0)
 		(unit 1)
 		(exclude_from_sim no)
@@
 		(dnp no)
 		(property "Reference" "#PWR083"
-			(at 212.09 30.48 0)
+			(at 173.99 139.7 0)
 			(effects
 				(font
@@
 		)
 		(property "Value" "+24V"
-			(at 209.296 22.606 0)
+			(at 171.196 131.826 0)
 			(effects
 				(font
@@
 		)
 		(property "Footprint" ""
-			(at 212.09 26.67 0)
+			(at 173.99 135.89 0)
 			(effects
 				(font
@@
 		)
 		(property "Datasheet" ""
-			(at 212.09 26.67 0)
+			(at 173.99 135.89 0)
 			(effects
 				(font
@@
 		)
 		(property "Description" "Power symbol creates a global label with name \"+12V\""
-			(at 212.09 26.67 0)
+			(at 173.99 135.89 0)
 			(effects
 				(font
@@
 	(symbol
 		(lib_id "power:GND")
-		(at 215.9 62.23 0)
+		(at 215.9 72.39 0)
 		(unit 1)
 		(exclude_from_sim no)
@@
 		(fields_autoplaced yes)
 		(property "Reference" "#PWR04"
-			(at 215.9 68.58 0)
+			(at 215.9 78.74 0)
 			(effects
 				(font
@@
 		)
 		(property "Value" "GND"
-			(at 215.9 67.31 0)
+			(at 215.9 77.47 0)
 			(effects
 				(font
@@
 		)
 		(property "Footprint" ""
-			(at 215.9 62.23 0)
+			(at 215.9 72.39 0)
 			(effects
 				(font
@@
 		)
 		(property "Datasheet" ""
-			(at 215.9 62.23 0)
+			(at 215.9 72.39 0)
 			(effects
 				(font
@@
 		)
 		(property "Description" "Power symbol creates a global label with name \"GND\" , ground"
-			(at 215.9 62.23 0)
+			(at 215.9 72.39 0)
 			(effects
 				(font
@@
 	(symbol
 		(lib_id "Device:Fuse")
-		(at 223.52 57.15 90)
+		(at 223.52 67.31 90)
 		(unit 1)
 		(exclude_from_sim no)
@@
 		(dnp no)
 		(property "Reference" "F1"
-			(at 223.52 52.324 90)
+			(at 223.52 62.484 90)
 			(effects
 				(font
@@
 		)
 		(property "Value" "1A"
-			(at 223.52 54.864 90)
+			(at 223.52 65.024 90)
 			(effects
 				(font
@@
 			)
 		)
-		(property "Footprint" ""
-			(at 223.52 58.928 90)
+		(property "Footprint" "Fuse:Fuse_0805_2012Metric"
+			(at 223.52 69.088 90)
 			(effects
 				(font
@@
 		)
 		(property "Datasheet" "~"
-			(at 223.52 57.15 0)
+			(at 223.52 67.31 0)
 			(effects
 				(font
@@
 		)
 		(property "Description" "Fuse"
-			(at 223.52 57.15 0)
+			(at 223.52 67.31 0)
+			(effects
+				(font
+					(size 1.27 1.27)
+				)
+				(hide yes)
+			)
+		)
+		(property "P/N" "MFU0805FF01000P500"
+			(at 223.52 67.31 90)
 			(effects
 				(font
@@
 	(symbol
 		(lib_id "power:+12V")
-		(at 231.14 57.15 0)
+		(at 231.14 67.31 0)
 		(unit 1)
 		(exclude_from_sim no)
@@
 		(dnp no)
 		(property "Reference" "#PWR0117"
-			(at 231.14 60.96 0)
+			(at 231.14 71.12 0)
 			(effects
 				(font
@@
 		)
 		(property "Value" "+24V"
-			(at 228.346 53.086 0)
+			(at 228.346 63.246 0)
 			(effects
 				(font
@@
 		)
 		(property "Footprint" ""
-			(at 231.14 57.15 0)
+			(at 231.14 67.31 0)
 			(effects
 				(font
@@
 		)
 		(property "Datasheet" ""
-			(at 231.14 57.15 0)
+			(at 231.14 67.31 0)
 			(effects
 				(font
@@
 		)
 		(property "Description" "Power symbol creates a global label with name \"+12V\""
-			(at 231.14 57.15 0)
+			(at 231.14 67.31 0)
 			(effects
 				(font
@@
 	(symbol
 		(lib_id "UTSVT_Connectors:CarLVPowerConnector")
-		(at 208.28 59.69 0)
+		(at 208.28 69.85 0)
 		(unit 1)
 		(exclude_from_sim no)
@@
 		(dnp no)
 		(property "Reference" "J2"
-			(at 207.645 54.61 0)
+			(at 207.645 64.77 0)
 			(effects
 				(font
@@
 		)
 		(property "Value" "Display Breakout"
-			(at 209.55 52.07 0)
+			(at 209.55 62.23 0)
 			(effects
 				(font
@@
 		)
 		(property "Footprint" "UTSVT_Connectors:Molex_Nano-Fit_105309-xx02_1x02_P2.50mm_Vertical"
-			(at 208.28 59.69 0)
+			(at 208.28 69.85 0)
 			(effects
 				(font
@@
 		)
 		(property "Datasheet" ""
-			(at 208.28 59.69 0)
+			(at 208.28 69.85 0)
 			(effects
 				(font
@@
 		)
 		(property "Description" "Connector for the car's 24V power bus"
-			(at 208.28 59.69 0)
+			(at 208.28 69.85 0)
 			(effects
 				(font
@@
 		)
 		(property "P/N" ""
-			(at 208.28 59.69 0)
+			(at 208.28 69.85 0)
 			(effects
 				(font
@@
 	(symbol
 		(lib_id "power:+5V")
-		(at 219.71 26.67 0)
+		(at 181.61 135.89 0)
 		(unit 1)
 		(exclude_from_sim no)
@@
 		(dnp no)
 		(property "Reference" "#PWR084"
-			(at 219.71 30.48 0)
+			(at 181.61 139.7 0)
 			(effects
 				(font
@@
 		)
 		(property "Value" "+5V"
-			(at 219.456 22.352 0)
+			(at 181.356 131.572 0)
 			(effects
 				(font
@@
 		)
 		(property "Footprint" ""
-			(at 219.71 26.67 0)
+			(at 181.61 135.89 0)
 			(effects
 				(font
@@
 		)
 		(property "Datasheet" ""
-			(at 219.71 26.67 0)
+			(at 181.61 135.89 0)
 			(effects
 				(font
@@
 		)
 		(property "Description" "Power symbol creates a global label with name \"+5V\""
-			(at 219.71 26.67 0)
+			(at 181.61 135.89 0)
 			(effects
 				(font

Commit message: I hate my life
Parts:
- removed C26: 22n, Capacitor_SMD:C_0603_1608Metric, symbol Device:C
- removed F1: 1A, Fuse:Fuse_0805_2012Metric, symbol Device:Fuse
- removed J1: CarLVPowerConnector, UTSVT_Connectors:Molex_Nano-Fit_105309-xx02_1x02_P2.50mm_Vertical, symbol UTSVT_Connectors:CarLVPowerConnector
- removed Q1: PSMN8R5-40MSDX, UTSVT_Power_SP:PSMN8R5-40MSDX, symbol UTSVT_Power:PSMN8R5-40MSDX
- removed Z2: SMAF4751A-TP, UTSVT_Passives:SODFL5026X125N, symbol UTSVT_Power:SMAF4749A-TP
- added C3: 0.1u, Capacitor_SMD:C_0603_1608Metric_Pad1.08x0.95mm_HandSolder, symbol Device:C
- added F1: 3568, Controls_Pi:FUSE_3568, symbol 3568:3568
- added J1: CarLVPowerConnector, UTSVT_Connectors:Molex_Nano-Fit_105309-xx02_1x02_P2.50mm_Vertical, symbol utsvt_connectors:CarLVPowerConnector
- added Q1: PSMN8R5-40MSDX, UTSVT_Power:PSMN8R5-40MSDX, symbol utsvt_power:PSMN8R5-40MSDX
- C18, C19, C27, C6, C61, C8, C9: footprint Capacitor_SMD:C_0603_1608Metric -> Capacitor_SMD:C_0805_2012Metric_Pad1.18x1.45mm_HandSolder
- C5, C56, C59, C60, C7: footprint Capacitor_SMD:C_0603_1608Metric -> Capacitor_SMD:C_0603_1608Metric_Pad1.08x0.95mm_HandSolder
- C58: footprint Capacitor_SMD:C_0805_2012Metric -> Capacitor_SMD:C_0805_2012Metric_Pad1.18x1.45mm_HandSolder
- D7, D9: footprint LED_SMD:LED_0603_1608Metric -> LED_SMD:LED_0603_1608Metric_Pad1.05x0.95mm_HandSolder
- R100, R13, R14, R44, R45: footprint Resistor_SMD:R_0603_1608Metric -> Resistor_SMD:R_0603_1608Metric_Pad0.98x0.95mm_HandSolder
- R30, R31: footprint Resistor_SMD:R_0805_2012Metric -> Resistor_SMD:R_0805_2012Metric_Pad1.20x1.40mm_HandSolder
Connections:
- net +24V: now also F1.2, F1.4, Q1.1 (S_1), Q1.2 (S_2), Q1.3 (S_3)
- net GND: now also C3.1, J1.2 (GND)
- net LV+: now also C3.2, J1.1 (+24V), Q1.10 (D_6), Q1.11 (D_7), Q1.5 (D_1), Q1.6 (D_2), Q1.7 (D_3), Q1.8 (D_4), Q1.9 (D_5)
- net at IC3.6 (GATE): now also Q1.4 (G)
- net at J2.1 (+24V): now also F1.1, F1.3
Other:
- note added: "From VCU"

Commit message: frank
Parts:
- removed Q1: PSMN8R5-40MSDX, UTSVT_Power:PSMN8R5-40MSDX, symbol utsvt_power:PSMN8R5-40MSDX
- added Q2, Q3: NVMFWS1D7N04XMT1G, Controls_Pi:NVMFWS3D0P04M8LT1G, symbol NVMFWS1D7N04XMT1G:NVMFWS1D7N04XMT1G
Connections:
- net +24V: now also Q3.5, Q3.6, Q3.7, Q3.8, Q3.9
- net LV+: now also Z1.1 (K), Q2.5, Q2.6, Q2.7, Q2.8, Q2.9
- net RPP_EN: no longer Z1.1 (K)
- net at IC3.6 (GATE): now also Q2.4, Q3.4
- new net: Q2.1, Q2.2, Q2.3, Q3.1, Q3.2, Q3.3
Other:
- moved on the sheet: C18, C27, C3, J1, Z1

Commit message: frink
Parts:
- C27: value 220u -> 10u
Changed lines of the file:
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@@
 		(fields_autoplaced yes)
 		(property "Reference" "C27"
-			(at 120.015 40.6399 0)
+			(at 120.65 40.6399 0)
 			(effects
 				(font
@@
 			)
 		)
-		(property "Value" "220u"
-			(at 120.015 43.1799 0)
+		(property "Value" "10u"
+			(at 120.65 43.1799 0)
 			(effects
 				(font

Commit message: lak
Parts:
- removed R100: 10k, Resistor_SMD:R_0603_1608Metric_Pad0.98x0.95mm_HandSolder, symbol Device:R_US
Connections:
- net RPP_EN is gone; now on net LV+: C18.2, C19.1, IC3.1 (EN/UVLO), IC3.5 (VS)
- net +24V: no longer IC3.8 (SRC)
- net at Q2.1, Q2.2, Q2.3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: now also IC3.8 (SRC)
Changed lines of the file:
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@@
 	)
 	(junction
-		(at 110.49 35.56)
-		(diameter 0)
-		(color 0 0 0 0)
-	)
-	(junction
 		(at 86.36 35.56)
 		(diameter 0)
@@
 	(wire
 		(pts
-			(xy 63.5 52.07) (xy 63.5 35.56)
+			(xy 63.5 35.56) (xy 63.5 62.23)
 		)
 		(stroke
@@
 	(wire
 		(pts
-			(xy 110.49 35.56) (xy 110.49 50.8)
-		)
-		(stroke
-			(width 0)
-			(type default)
-		)
-	)
-	(wire
-		(pts
 			(xy 107.95 132.08) (xy 107.95 139.7)
 		)
@@
 	(wire
 		(pts
-			(xy 86.36 50.8) (xy 110.49 50.8)
-		)
-		(stroke
-			(width 0)
-			(type default)
-		)
-	)
-	(wire
-		(pts
 			(xy 29.21 132.08) (xy 35.56 132.08)
 		)
@@
 	(wire
 		(pts
-			(xy 110.49 35.56) (xy 116.84 35.56)
+			(xy 105.41 35.56) (xy 116.84 35.56)
 		)
 		(stroke
@@
 	(wire
 		(pts
+			(xy 86.36 38.1) (xy 86.36 54.61)
+		)
+		(stroke
+			(width 0)
+			(type default)
+		)
+	)
+	(wire
+		(pts
 			(xy 80.01 44.45) (xy 76.2 44.45)
 		)
@@
 	(wire
 		(pts
-			(xy 105.41 35.56) (xy 110.49 35.56)
-		)
-		(stroke
-			(width 0)
-			(type default)
-		)
-	)
-	(wire
-		(pts
 			(xy 116.84 35.56) (xy 125.73 35.56)
 		)
@@
 	(wire
 		(pts
-			(xy 63.5 59.69) (xy 63.5 62.23)
-		)
-		(stroke
-			(width 0)
-			(type default)
-		)
-	)
-	(wire
-		(pts
 			(xy 35.56 132.08) (xy 35.56 130.81)
 		)
@@
 	(wire
 		(pts
-			(xy 86.36 54.61) (xy 86.36 50.8)
-		)
-		(stroke
-			(width 0)
-			(type default)
-		)
-	)
-	(wire
-		(pts
 			(xy 105.41 35.56) (xy 105.41 38.1)
 		)
@@
 					(unit 1)
 				)
-			)
-		)
-	)
-	(symbol
-		(lib_id "Device:R_US")
-		(at 63.5 55.88 0)
-		(unit 1)
-		(exclude_from_sim no)
-		(in_bom yes)
-		(on_board yes)
-		(dnp no)
-		(fields_autoplaced yes)
-		(property "Reference" "R100"
-			(at 65.405 54.6099 0)
-			(effects
-				(font
-					(size 1.27 1.27)
-				)
-				(justify left)
-			)
-		)
-		(property "Value" "10k"
-			(at 65.405 57.1499 0)
-			(effects
-				(font
-					(size 1.27 1.27)
-				)
-				(justify left)
-			)
-		)
-		(property "Footprint" "Resistor_SMD:R_0603_1608Metric_Pad0.98x0.95mm_HandSolder"
-			(at 64.516 56.134 90)
-			(effects
-				(font
-					(size 1.27 1.27)
-				)
-				(hide yes)
-			)
-		)
-		(property "Datasheet" "~"
-			(at 63.5 55.88 0)
-			(effects
-				(font
-					(size 1.27 1.27)
-				)
-				(hide yes)
-			)
-		)
-		(property "Description" "Resistor, US symbol"
-			(at 63.5 55.88 0)
-			(effects
-				(font
-					(size 1.27 1.27)
-				)
-				(hide yes)
-			)
-		)
-		(pin "1"
-		)
-		(pin "2"
-		)
-		(instances
-			(project "PiBoard"
-				(path "/e4d65698-b8ec-4bf6-9f2b-a5010377155a/0c1fd794-8ba7-4f58-ad3e-1ee234c84a43"
-					(reference "R100")
-					(unit 1)
-				)

Commit message: chang
Parts:
- Z1: P/N (none) -> SMAF4751A
Changed lines of the file:
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@@
+			)
+		)
+		(property "P/N" "SMAF4751A"
+			(at 44.45 33.02 90)
+			(effects
+				(font
+					(size 1.27 1.27)
+				)
+				(hide yes)
 			)
 		)

Commit message: P/Ns
Parts:
- C18: value 1u -> 1uF; P/N (none) -> MLASU168SB5105KTNA01
- C19: value 220n -> 220nF; P/N (none) -> MSASU168SB7224KTNB25
- C27: value 10u -> 10uF; P/N (none) -> GRM21BR61H106KE43K
- C3: value 0.1u -> 100n; P/N (none) -> MLASH168SB7104KTNA01
- C5, C7: P/N C0805C104M5RACTU -> MLASH168SB7104KTNA01
- C56: value 10n -> 10nF; P/N C0805C103J5RACTU -> MSASH168SB5103KTNA01
- C58: P/N 0805W106K500CC -> GRM21BR61H106KE43K
- C59: value 2.7n -> 2.7nF; P/N VJ0805A272JXAAT -> 08051C272J4Z2A
- C6: P/N C0805C104M5RACTU -> GRM21BR61H106KE43K
- C60: value 33p -> 33pF; P/N C0805C330J5RACTU -> C0603X330M1HACTU
- C61, C8, C9: value 22u -> 22uF; P/N CL21A226KQCLRNC -> C2012X5R1V226M125AC
- D7, D9: P/N APTD2012LCGCK -> 150060VS55040
- F1: P/N (none) -> 3568
- IC3: P/N (none) -> LM74502HDDFR
- L2: value 4.7 u -> 4.7uH
- Q2, Q3: P/N (none) -> NVMFWS1D7N04XMT1G
- R13: P/N (none) -> CRCW060310K0FKEI
- R14: P/N (none) -> MCT06030C2003FP500
- R31: P/N RC0805FR-0752K3L -> RMCF0805FT52K3
- R32: P/N CRCW080510K0FKEAC -> AC0805DR-0710KL
- R44: value 10k -> 1.5k; footprint Resistor_SMD:R_0603_1608Metric_Pad0.98x0.95mm_HandSolder -> Resistor_SMD:R_0805_2012Metric_Pad1.20x1.40mm_HandSolder; P/N CRCW08055K00FKTA -> ERJ-UP6F1501V
- R45: value 1.5k -> 200; P/N SDR10EZPF1501 -> SG73S1JTTD2000F
- Z1: value SMAF4751A-TP -> SMAF4759A-TP; P/N SMAF4751A -> SMAF4759A-TP
Other:
- note added: "R: ~1500 0.4W"
- note added: "R: ~200"
- note added: "fwd cur: ~20ma fwd volt: ~2V"
- note removed: "R: ~11000"
- note removed: "R: ~1500"
- note removed: "fwd cur: ~2ma fwd volt: ~2V"
