File: CarCAN.kicad_sch (KiCad schematic)
At the start: 18 parts, among them IC1 TCAN337DCNR, J6 CarCANConnector, J8 CarCANConnector, U13 CDSOT23-T24CAN, U14 MCP2515T-E/ST, Y4 8 MHz

Commit message: P/Ns
Parts:
- C11, C36, C37: P/N C0805C104M5RACTU -> MLASH168SB7104KTNA01
- C24, C25: P/N C0805C220J5HACTU -> 0603N220F101CT
- D4: P/N APTD2012LSURCK -> LS Q976.01-N1Q2-1
- R2: value 700 -> 100; P/N SDR10EZPF2200 -> CRCW0603100RFKEA
- R24: P/N CRCW1210120RFKEAHP -> CRCW0603120RFKEC
- R34, R35: P/N CRCW080510K0FKEAC -> CRCW060310K0FKEI
- R5: value 1000 -> 1k; P/N SDR10EZPF2200 -> CRCW06031K00FKEI
Changed lines of the file:
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@@
 			)
 		)
-		(property "P/N" "C0805C220J5HACTU"
+		(property "P/N" "0603N220F101CT"
+			(at 36.83 120.65 90)
+			(effects
+				(font
+					(size 1.27 1.27)
+				)
+				(hide yes)
+			)
+		)
+		(property "Data" ""
 			(at 36.83 120.65 90)
 			(effects
@@
 			)
 		)
-		(property "P/N" "C0805C104M5RACTU"
+		(property "P/N" "MLASH168SB7104KTNA01 "
+			(at 106.68 129.54 0)
+			(effects
+				(font
+					(size 1.27 1.27)
+				)
+				(hide yes)
+			)
+		)
+		(property "Data" ""
 			(at 106.68 129.54 0)
 			(effects
@@
 			)
 		)
-		(property "P/N" "APTD2012LSURCK "
+		(property "P/N" "LS Q976.01-N1Q2-1 "
 			(at 262.89 113.03 0)
 			(effects
@@
 			)
 		)
+		(property "Data" ""
+			(at 262.89 113.03 90)
+			(effects
+				(font
+					(size 1.27 1.27)
+				)
+				(hide yes)
+			)
+		)
 		(pin "1"
 		)
@@
 			)
 		)
-		(property "P/N" "CRCW1210120RFKEAHP"
+		(property "P/N" "CRCW0603120RFKEC  "
 			(at 208.28 115.57 0)
+			(effects
+				(font
+					(size 1.27 1.27)
+				)
+				(hide yes)
+			)
+		)
+		(property "Data" ""
+			(at 208.28 115.57 90)
 			(effects
 				(font
@@
 			)
 		)
-		(property "P/N" "C0805C220J5HACTU"
+		(property "P/N" "0603N220F101CT"
+			(at 36.83 110.49 90)
+			(effects
+				(font
+					(size 1.27 1.27)
+				)
+				(hide yes)
+			)
+		)
+		(property "Data" ""
 			(at 36.83 110.49 90)
 			(effects
@@
 			)
 		)
+		(property "Data" ""
+			(at 233.68 99.06 0)
+			(effects
+				(font
+					(size 1.27 1.27)
+				)
+				(hide yes)
+			)
+		)
 		(pin "2"
 		)
@@
 			)
 		)
-		(property "Value" "1000"
+		(property "Value" "1k"
 			(at 108.458 120.523 0)
 			(effects
@@
 			)
 		)
-		(property "P/N" "SDR10EZPF2200"
+		(property "P/N" "CRCW06031K00FKEI  "
+			(at 106.68 119.38 0)
+			(effects
+				(font
+					(size 1.27 1.27)
+				)
+				(hide yes)
+			)
+		)
+		(property "Data" ""
 			(at 106.68 119.38 0)
 			(effects
@@
 			)
 		)
-		(property "P/N" "CRCW080510K0FKEAC"
+		(property "P/N" "CRCW060310K0FKEI  "
+			(at 193.04 99.06 0)
+			(effects
+				(font
+					(size 1.27 1.27)
+				)
+				(hide yes)
+			)
+		)
+		(property "Data" ""
 			(at 193.04 99.06 0)
 			(effects
@@
 		)
 		(property "P/N" ""
+			(at 200.66 120.65 0)
+			(effects
+				(font
+					(size 1.27 1.27)
+				)
+				(hide yes)
+			)
+		)
+		(property "Data" ""
 			(at 200.66 120.65 0)
 			(effects
@@
 			)
 		)
+		(property "Data" ""
+			(at 163.83 105.41 0)
+			(effects
+				(font
+					(size 1.27 1.27)
+				)
+				(hide yes)
+			)
+		)
 		(pin "2"
 		)
@@
 			)
 		)
+		(property "Data" ""
+			(at 233.68 109.22 0)
+			(effects
+				(font
+					(size 1.27 1.27)
+				)
+				(hide yes)
+			)
+		)
 		(pin "2"
 		)
@@
 			)
 		)
+		(property "Data" ""
+			(at 226.06 121.92 0)
+			(effects
+				(font
+					(size 1.27 1.27)
+				)
+				(hide yes)
+			)
+		)
 		(pin "1"
 		)
@@
 			)
 		)
-		(property "P/N" "C0805C104M5RACTU"
+		(property "P/N" "MLASH168SB7104KTNA01 "
+			(at 100.33 87.63 0)
+			(effects
+				(font
+					(size 1.27 1.27)
+				)
+				(hide yes)
+			)
+		)
+		(property "Data" ""
 			(at 100.33 87.63 0)
 			(effects
@@
 			)
 		)
+		(property "Data" ""
+			(at 72.39 109.22 0)
+			(effects
+				(font
+					(size 1.27 1.27)
+				)
+				(hide yes)
+			)
+		)
 		(pin "6"
 		)
@@
 			)
 		)
+		(property "Data" ""
+			(at 44.45 115.57 90)
+			(effects
+				(font
+					(size 1.27 1.27)
+				)
+				(hide yes)
+			)
+		)
 		(pin "1"
 		)
@@
 			)
 		)
-		(property "Value" "700"
+		(property "Value" "100"
 			(at 264.668 105.283 0)
 			(effects
@@
 			)
 		)
-		(property "P/N" "SDR10EZPF2200"
+		(property "P/N" "CRCW0603100RFKEA"
+			(at 262.89 104.14 0)
+			(effects
+				(font
+					(size 1.27 1.27)
+				)
+				(hide yes)
+			)
+		)
+		(property "Data" ""
 			(at 262.89 104.14 0)
 			(effects
@@
 			)
 		)
-		(property "P/N" "CRCW080510K0FKEAC"
+		(property "P/N" "CRCW060310K0FKEI  "
 			(at 96.52 124.46 0)
+			(effects
+				(font
+					(size 1.27 1.27)
+				)
+				(hide yes)
+			)
+		)
+		(property "Data" ""
+			(at 96.52 124.46 90)
 			(effects
 				(font
@@
 			)
 		)
-		(property "P/N" "C0805C104M5RACTU"
+		(property "P/N" "MLASH168SB7104KTNA01 "
 			(at 149.86 115.57 0)
 			(effects
+				(font
+					(size 1.27 1.27)
+				)
+				(hide yes)
+			)
+		)
+		(property "Data" ""
+			(at 149.86 115.57 0)
+			(effects

Commit message: jlc shit
Parts:
- C11, C36, C37: JLC (none) -> C14663
- C24, C25: JLC (none) -> C1653
- D4: JLC (none) -> C2286
- IC1: JLC (none) -> C130129
- J6, J8, JP1: JLC (none) -> N/A
- R2: JLC (none) -> C22775
- R24: JLC (none) -> C22787
- R34, R35: JLC (none) -> C25804
- R5: JLC (none) -> C21190
- U13: JLC (none) -> C2959841
- U14: JLC (none) -> C627064
- Y4: JLC (none) -> C144380
Changed lines of the file:
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@@
+			)
+		)
+		(property "JLC" "C1653"
+			(at 36.83 120.65 90)
+			(effects
+				(font
+					(size 1.27 1.27)
+				)
+				(hide yes)
 			)
 		)
@@
 			)
 		)
+		(property "JLC" "C14663"
+			(at 106.68 129.54 0)
+			(effects
+				(font
+					(size 1.27 1.27)
+				)
+				(hide yes)
+			)
+		)
 		(pin "1"
 		)
@@
 			)
 		)
+		(property "JLC" "C2286"
+			(at 262.89 113.03 90)
+			(effects
+				(font
+					(size 1.27 1.27)
+				)
+				(hide yes)
+			)
+		)
 		(pin "1"
 		)
@@
 			)
 		)
+		(property "JLC" "C22787"
+			(at 208.28 115.57 90)
+			(effects
+				(font
+					(size 1.27 1.27)
+				)
+				(hide yes)
+			)
+		)
 		(pin "1"
 		)
@@
 		)
 		(property "Data" ""
+			(at 36.83 110.49 90)
+			(effects
+				(font
+					(size 1.27 1.27)
+				)
+				(hide yes)
+			)
+		)
+		(property "JLC" "C1653"
 			(at 36.83 110.49 90)
 			(effects
@@
 			)
 		)
+		(property "JLC" "N/A"
+			(at 233.68 99.06 0)
+			(effects
+				(font
+					(size 1.27 1.27)
+				)
+				(hide yes)
+			)
+		)
 		(pin "2"
 		)
@@
 		)
 		(property "Data" ""
+			(at 106.68 119.38 0)
+			(effects
+				(font
+					(size 1.27 1.27)
+				)
+				(hide yes)
+			)
+		)
+		(property "JLC" "C21190"
 			(at 106.68 119.38 0)
 			(effects
@@
 			)
 		)
+		(property "JLC" "C25804"
+			(at 193.04 99.06 0)
+			(effects
+				(font
+					(size 1.27 1.27)
+				)
+				(hide yes)
+			)
+		)
 		(pin "1"
 		)
@@
 		)
 		(property "Data" ""
+			(at 200.66 120.65 0)
+			(effects
+				(font
+					(size 1.27 1.27)
+				)
+				(hide yes)
+			)
+		)
+		(property "JLC" "N/A"
 			(at 200.66 120.65 0)
 			(effects
@@
 			)
 		)
+		(property "JLC" "C130129"
+			(at 163.83 105.41 0)
+			(effects
+				(font
+					(size 1.27 1.27)
+				)
+				(hide yes)
+			)
+		)
 		(pin "2"
 		)
@@
 			)
 		)
+		(property "JLC" "N/A"
+			(at 233.68 109.22 0)
+			(effects
+				(font
+					(size 1.27 1.27)
+				)
+				(hide yes)
+			)
+		)
 		(pin "2"
 		)
@@
 			)
 		)
+		(property "JLC" "C2959841"
+			(at 226.06 121.92 0)
+			(effects
+				(font
+					(size 1.27 1.27)
+				)
+				(hide yes)
+			)
+		)
 		(pin "1"
 		)
@@
 			)
 		)
+		(property "JLC" "C14663"
+			(at 100.33 87.63 0)
+			(effects
+				(font
+					(size 1.27 1.27)
+				)
+				(hide yes)
+			)
+		)
 		(pin "1"
 		)
@@
 			)
 		)
+		(property "JLC" "C627064"
+			(at 72.39 109.22 0)
+			(effects
+				(font
+					(size 1.27 1.27)
+				)
+				(hide yes)
+			)
+		)
 		(pin "6"
 		)
@@
 			)
 		)
+		(property "JLC" "C144380"
+			(at 44.45 115.57 90)
+			(effects
+				(font
+					(size 1.27 1.27)
+				)
+				(hide yes)
+			)
+		)
 		(pin "1"
 		)
@@
 		)
 		(property "Data" ""
+			(at 262.89 104.14 0)
+			(effects
+				(font
+					(size 1.27 1.27)
+				)
+				(hide yes)
+			)
+		)
+		(property "JLC" "C22775"
 			(at 262.89 104.14 0)
 			(effects
@@
 			)
 		)
+		(property "JLC" "C25804"
+			(at 96.52 124.46 90)
+			(effects
+				(font
+					(size 1.27 1.27)
+				)
+				(hide yes)
+			)
+		)
 		(pin "1"
 		)
@@
 			(at 149.86 115.57 0)
 			(effects
+				(font
+					(size 1.27 1.27)
+				)
+				(hide yes)
+			)
+		)
+		(property "JLC" "C14663"
+			(at 149.86 115.57 0)
+			(effects
