File: CM5_HighSpeed.kicad_sch (KiCad schematic)
At the start: 1 part

Commit message: Schem done? [plz full review], redoing layout
Other:
- note added: "Connectors"
- moved on the sheet: Module2B

Commit message: my life could not be worse right now
Other:
- note added: "USB"
- note removed: "USB-C"
Changed lines of the file:
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@@
 		)
 	)
-	(text "USB-C"
+	(text "USB\n"
 		(exclude_from_sim no)
 		(at 222.25 111.252 0)
@@
 			)
 		)
-		(property "Datasheet" "https://storage.raspberrypi.com/product-information/hawl3l9kl3xwo8tj8e2msztrus1n?response-content-disposition=inline%3B%20filename%3D%22RP-008180-DS-cm5-datasheet.pdf%22%3B%20filename%2A%3DUTF-8%27%27RP-008180-DS-cm5-datasheet.pdf&response-content-type=application%2Fpdf&X-Amz-Algorithm=AWS4-HMAC-SHA256&X-Amz-Credential=product-information%2F20251004%2Feu-west-1%2Fs3%2Faws4_request&X-Amz-Date=20251004T180850Z&X-Amz-Expires=172800&X-Amz-SignedHeaders=host&X-Amz-Signature=be9dd03b4fc44e5a401ffdce01adaaf5f36a0d9794c56bc665f3d3971a12888a"
+		(property "Datasheet" "https://pip-assets.raspberrypi.com/categories/944-raspberry-pi-compute-module-5/documents/RP-008180-DS-6-cm5-datasheet.pdf?disposition=inline"
 			(at 99.06 124.46 0)
 			(effects

Commit message: P/Ns
Parts:
- Module2: P/N (none) -> 10164227-1001A1RLF
Changed lines of the file:
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@@
+			)
+		)
+		(property "Data" ""
+			(at -43.18 97.79 0)
+			(effects
+				(font
+					(size 1.27 1.27)
+				)
+				(hide yes)
+			)
+		)
+		(property "P/N" "10164227-1001A1RLF"
+			(at -43.18 97.79 0)
+			(effects
+				(font
+					(size 1.27 1.27)
+				)
+				(hide yes)
 			)
 		)

Commit message: jlc shit
Parts:
- Module2: JLC (none) -> C6782225
Changed lines of the file:
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@@
+			)
+		)
+		(property "JLC" "C6782225"
+			(at -43.18 97.79 0)
+			(effects
+				(font
+					(size 1.27 1.27)
+				)
+				(hide yes)
 			)
 		)
